Commit message: Create Gazebo simulation package

File: src/solarbot_description/urdf/base/chassis.xacro (robot description, xacro)
@@ -1,41 +1,138 @@
 <?xml version="1.0"?>
 <robot xmlns:xacro="http://www.ros.org/wiki/xacro">
-  <!-- ============================= -->
-  <!-- Base Footprint                -->
-  <!-- ============================= -->
+  <!--
+    chassis.xacro
+    ─────────────────────────────────────────────────────────────────
+    Main chassis body: base_footprint, base_link.
+    Visuals represent the aluminium frame as seen on the real chassis:
+      • Central spine rail
+      • Front and rear top mounting plates
+      • Left and right side rails
+    Depends on: common/properties.xacro, common/materials.xacro
+  ─────────────────────────────────────────────────────────────────
+  -->
+  <!-- ── Inertia helper macros ─────────────────────────────── -->
+  <!-- Solid box: m=mass, lx/ly/lz=dimensions along each axis -->
+  <xacro:macro name="box_inertia" params="m lx ly lz">
+    <inertia
+      ixx="${m*(ly*ly + lz*lz)/12.0}"
+      ixy="0.0" ixz="0.0"
+      iyy="${m*(lx*lx + lz*lz)/12.0}"
+      iyz="0.0"
+      izz="${m*(lx*lx + ly*ly)/12.0}"/>
+  </xacro:macro>
+  <!-- Solid cylinder: m=mass, r=radius, h=height along spin axis -->
+  <xacro:macro name="cylinder_inertia" params="m r h">
+    <inertia
+      ixx="${m*(3.0*r*r + h*h)/12.0}"
+      ixy="0.0" ixz="0.0"
+      iyy="${m*(3.0*r*r + h*h)/12.0}"
+      iyz="0.0"
+      izz="${m*r*r/2.0}"/>
+  </xacro:macro>
+  <!-- ── base_footprint ────────────────────────────────────── -->
+  <!--
+    Projection of the robot onto the ground plane.
+    Nav2 and the localisation stack use this frame as the
+    reference for 2D pose (x, y, yaw).
+  -->
   <link name="base_footprint"/>
-  <!-- ============================= -->
-  <!-- Base Link                     -->
-  <!-- ============================= -->
-  <joint name="base_joint" type="fixed">
+  <joint name="base_footprint_joint" type="fixed">
     <parent link="base_footprint"/>
-    <child link="base_link"/>
-    <origin xyz="0 0 ${chassis_height/2}" rpy="0 0 0"/>
+    <child  link="base_link"/>
+    <!-- Raise base_link so the track bottoms sit at z=0 in the world -->
+    <origin xyz="0 0 ${base_z_above_ground}" rpy="0 0 0"/>
   </joint>
+  <!-- ── base_link ─────────────────────────────────────────── -->
+  <!--
+    Rigid chassis body.  The inertial block approximates the full
+    chassis as a solid box — good enough for simulation dynamics.
+    Visuals are broken into sub-boxes to resemble the real aluminium
+    frame visible in the chassis photo.
+  -->
   <link name="base_link">
+    <inertial>
+      <origin xyz="0 0 0" rpy="0 0 0"/>
+      <mass value="${chassis_mass}"/>
+      <xacro:box_inertia
+        m="${chassis_mass}"
+        lx="${track_full_length}"
+        ly="${motor_shaft_length}"
+        lz="${track_pod_height}"/>
+    </inertial>
+    <!-- ── Visual: central spine rail ── -->
     <visual>
-      <origin xyz="0 0 0"/>
+      <origin xyz="0 0 0" rpy="0 0 0"/>
       <geometry>
-        <box size="${chassis_length} ${chassis_width} ${chassis_height}"/>
+        <box size="${chassis_rail_length}
+                   ${chassis_rail_width}
+                   ${chassis_rail_height}"/>
       </geometry>
       <material name="silver"/>
     </visual>
     <collision>
-      <origin xyz="0 0 0"/>
+      <origin xyz="0 0 0" rpy="0 0 0"/>
       <geometry>
-        <box size="${chassis_length} ${chassis_width} ${chassis_height}"/>
+        <box size="${chassis_rail_length}
+                   ${chassis_rail_width}
+                   ${chassis_rail_height}"/>
       </geometry>
     </collision>
-    <inertial>
-      <origin xyz="0 0 0"/>
-      <mass value="${robot_mass}"/>
-      <inertia
-        ixx="0.05"
-        ixy="0.0"
-        ixz="0.0"
-        iyy="0.05"
-        iyz="0.0"
-        izz="0.08"/>
-    </inertial>
+    <!-- ── Visual: front top plate ── -->
+    <visual>
+      <origin xyz="${plate_length} 0 ${plate_z}" rpy="0 0 0"/>
+      <geometry>
+        <box size="${plate_length}
+                   ${plate_width}
+                   ${plate_thickness}"/>
+      </geometry>
+      <material name="silver"/>
+    </visual>
+    <collision>
+      <origin xyz="${plate_length} 0 ${plate_z}" rpy="0 0 0"/>
+      <geometry>
+        <box size="${plate_length}
+                   ${plate_width}
+                   ${plate_thickness}"/>
+      </geometry>
+    </collision>
+    <!-- ── Visual: rear top plate ── -->
+    <visual>
+      <origin xyz="${-plate_length} 0 ${plate_z}" rpy="0 0 0"/>
+      <geometry>
+        <box size="${plate_length}
+                   ${plate_width}
+                   ${plate_thickness}"/>
+      </geometry>
+      <material name="silver"/>
+    </visual>
+    <collision>
+      <origin xyz="${-plate_length} 0 ${plate_z}" rpy="0 0 0"/>
+      <geometry>
+        <box size="${plate_length}
+                   ${plate_width}
+                   ${plate_thickness}"/>
+      </geometry>
+    </collision>
+    <!-- ── Visual: left side rail ── -->
+    <visual>
+      <origin xyz="0 ${side_rail_y} ${side_rail_z}" rpy="0 0 0"/>
+      <geometry>
+        <box size="${side_rail_length}
+                   ${side_rail_width}
+                   ${side_rail_height}"/>
+      </geometry>
+      <material name="silver"/>
+    </visual>
+    <!-- ── Visual: right side rail ── -->
+    <visual>
+      <origin xyz="0 ${-side_rail_y} ${side_rail_z}" rpy="0 0 0"/>
+      <geometry>
+        <box size="${side_rail_length}
+                   ${side_rail_width}
+                   ${side_rail_height}"/>
+      </geometry>
+      <material name="silver"/>
+    </visual>
   </link>
 </robot>

File: src/solarbot_description/urdf/base/tracks.xacro (robot description, xacro)
@@ -1,56 +1,146 @@
 <?xml version="1.0"?>
 <robot xmlns:xacro="http://www.ros.org/wiki/xacro">
-  <!-- ========================================================= -->
-  <!-- Track Module Macro                                        -->
-  <!-- ========================================================= -->
-  <xacro:macro name="track_module" params="name x y">
-    <joint name="${name}_joint" type="fixed">
-      <parent link="base_link"/>
-      <child link="${name}_track_link"/>
-      <origin xyz="${x} ${y} 0" rpy="0 0 0"/>
-    </joint>
+  <!--
+    tracks.xacro
+    ─────────────────────────────────────────────────────────────────
+    Track pods (4 × fixed visual boxes), motor shaft visuals (2),
+    and virtual wheel joints (2) for diff_drive_controller.
+    Why virtual wheels?
+      diff_drive_controller requires continuous revolute joints to
+      send velocity commands to.  The 4 track pod joints are fixed
+      (they are rigid visual elements — tracks don't steer or pivot).
+      We therefore add two invisible virtual wheel links — one at
+      the lateral centre of each track side — that the controller
+      can command.  The Arduino firmware then mirrors each side's
+      command to both physical motors on that side.
+    Joint names used here MUST match diff_drive_controller config:
+      left_wheel_joint   ← left track
+      right_wheel_joint  ← right track
+    Depends on: common/properties.xacro, common/materials.xacro
+  ─────────────────────────────────────────────────────────────────
+  -->
+  <!-- ══════════════════════════════════════════════════════════ -->
+  <!-- Macro: single track pod (box visual, fixed joint)        -->
+  <!-- ══════════════════════════════════════════════════════════ -->
+  <xacro:macro name="track_pod" params="name x y">
     <link name="${name}_track_link">
+      <inertial>
+        <origin xyz="0 0 0" rpy="0 0 0"/>
+        <mass value="${track_pod_mass}"/>
+        <inertia
+          ixx="${track_pod_mass*(track_pod_width*track_pod_width  + track_pod_height*track_pod_height)/12.0}"
+          ixy="0" ixz="0"
+          iyy="${track_pod_mass*(track_pod_length*track_pod_length + track_pod_height*track_pod_height)/12.0}"
+          iyz="0"
+          izz="${track_pod_mass*(track_pod_length*track_pod_length + track_pod_width*track_pod_width)/12.0}"/>
+      </inertial>
       <visual>
+        <origin xyz="0 0 0" rpy="0 0 0"/>
         <geometry>
-          <box size="${track_length} ${track_width} ${track_height}"/>
+          <box size="${track_pod_length}
+                     ${track_pod_width}
+                     ${track_pod_height}"/>
         </geometry>
-        <material name="dark_gray"/>
+        <material name="black"/>
       </visual>
       <collision>
+        <origin xyz="0 0 0" rpy="0 0 0"/>
         <geometry>
-          <box size="${track_length} ${track_width} ${track_height}"/>
+          <box size="${track_pod_length}
+                     ${track_pod_width}
+                     ${track_pod_height}"/>
         </geometry>
       </collision>
+    </link>
+    <!-- Fixed joint: track pod is rigidly attached to chassis -->
+    <joint name="${name}_track_joint" type="fixed">
+      <parent link="base_link"/>
+      <child  link="${name}_track_link"/>
+      <origin xyz="${x} ${y} ${track_z_offset}" rpy="0 0 0"/>
+    </joint>
+  </xacro:macro>
+  <!-- ══════════════════════════════════════════════════════════ -->
+  <!-- Macro: virtual wheel link + continuous joint              -->
+  <!-- ══════════════════════════════════════════════════════════ -->
+  <xacro:macro name="virtual_wheel" params="name y_offset">
+    <!--
+      No visual or collision — purely a control artifact.
+      Placed at the lateral centre of each track at ground-contact
+      height (z = -wheel_radius from base_link = ground level).
+    -->
+    <link name="${name}_virtual_wheel_link">
       <inertial>
-        <mass value="0.4"/>
-        <origin xyz="0 0 0"/>
+        <origin xyz="0 0 0" rpy="0 0 0"/>
+        <mass value="${virtual_wheel_mass}"/>
         <inertia
-          ixx="0.001"
-          ixy="0"
-          ixz="0"
-          iyy="0.001"
+          ixx="${virtual_wheel_mass*(3.0*wheel_radius*wheel_radius + wheel_width*wheel_width)/12.0}"
+          ixy="0" ixz="0"
+          iyy="${virtual_wheel_mass*(3.0*wheel_radius*wheel_radius + wheel_width*wheel_width)/12.0}"
           iyz="0"
-          izz="0.001"/>
+          izz="${virtual_wheel_mass*wheel_radius*wheel_radius/2.0}"/>
       </inertial>
     </link>
+    <joint name="${name}_wheel_joint" type="continuous">
+      <parent link="base_link"/>
+      <child  link="${name}_virtual_wheel_link"/>
+      <!-- Centred longitudinally (x=0), at track y, at contact height -->
+      <origin xyz="0 ${y_offset} ${-wheel_radius}" rpy="0 0 0"/>
+      <!-- Standard diff-drive: wheel spins around the lateral (y) axis -->
+      <axis xyz="0 1 0"/>
+      <dynamics damping="0.01" friction="0.1"/>
+    </joint>
   </xacro:macro>
-  <!-- ========================================================= -->
-  <!-- Instantiate the four track modules                        -->
-  <!-- ========================================================= -->
-  <xacro:track_module
-      name="front_left"
-      x="${front_track_x}"
-      y="${left_track_y}"/>
-  <xacro:track_module
-      name="front_right"
-      x="${front_track_x}"
-      y="${right_track_y}"/>
-  <xacro:track_module
-      name="rear_left"
-      x="${rear_track_x}"
-      y="${left_track_y}"/>
-  <xacro:track_module
-      name="rear_right"
-      x="${rear_track_x}"
-      y="${right_track_y}"/>
+  <!-- ══════════════════════════════════════════════════════════ -->
+  <!-- Instantiate four track pods                              -->
+  <!-- ══════════════════════════════════════════════════════════ -->
+  <xacro:track_pod name="front_left"
+                   x="${track_front_x}"
+                   y="${track_y_offset}"/>
+  <xacro:track_pod name="rear_left"
+                   x="${track_rear_x}"
+                   y="${track_y_offset}"/>
+  <xacro:track_pod name="front_right"
+                   x="${track_front_x}"
+                   y="${-track_y_offset}"/>
+  <xacro:track_pod name="rear_right"
+                   x="${track_rear_x}"
+                   y="${-track_y_offset}"/>
+  <!-- ══════════════════════════════════════════════════════════ -->
+  <!-- Motor shaft visuals (fixed, cosmetic only)               -->
+  <!-- ══════════════════════════════════════════════════════════ -->
+  <link name="front_motor_link">
+    <visual>
+      <!-- rpy rotates the cylinder to lie along the y-axis (lateral) -->
+      <origin xyz="0 0 0" rpy="1.5708 0 0"/>
+      <geometry>
+        <cylinder radius="${motor_radius}" length="${motor_shaft_length}"/>
+      </geometry>
+      <material name="silver"/>
+    </visual>
+  </link>
+  <joint name="front_motor_joint" type="fixed">
+    <parent link="base_link"/>
+    <child  link="front_motor_link"/>
+    <origin xyz="${motor_front_x} 0 ${motor_z}" rpy="0 0 0"/>
+  </joint>
+  <link name="rear_motor_link">
+    <visual>
+      <origin xyz="0 0 0" rpy="1.5708 0 0"/>
+      <geometry>
+        <cylinder radius="${motor_radius}" length="${motor_shaft_length}"/>
+      </geometry>
+      <material name="silver"/>
+    </visual>
+  </link>
+  <joint name="rear_motor_joint" type="fixed">
+    <parent link="base_link"/>
+    <child  link="rear_motor_link"/>
+    <origin xyz="${-motor_front_x} 0 ${motor_z}" rpy="0 0 0"/>
+  </joint>
+  <!-- ══════════════════════════════════════════════════════════ -->
+  <!-- Two virtual wheel joints (one per track side)            -->
+  <!-- These are what diff_drive_controller actually commands.  -->
+  <!-- ══════════════════════════════════════════════════════════ -->
+  <xacro:virtual_wheel name="left"  y_offset="${track_y_offset}"/>
+  <xacro:virtual_wheel name="right" y_offset="${-track_y_offset}"/>
 </robot>

File: src/solarbot_description/urdf/common/materials.xacro (robot description, xacro)
@@ -1,30 +1,32 @@
 <?xml version="1.0"?>
 <robot xmlns:xacro="http://www.ros.org/wiki/xacro">
-  <!-- ============================= -->
-  <!-- Materials                     -->
-  <!-- ============================= -->
+  <!--
+    materials.xacro
+    All colour definitions. Reference by name everywhere else.
+  -->
+  <material name="silver">
+    <color rgba="0.75 0.75 0.72 1.0"/>
+  </material>
   <material name="black">
-    <color rgba="0.10 0.10 0.10 1.0"/>
+    <color rgba="0.05 0.05 0.05 1.0"/>
   </material>
   <material name="dark_gray">
-    <color rgba="0.25 0.25 0.25 1.0"/>
+    <color rgba="0.15 0.15 0.15 1.0"/>
   </material>
-  <material name="light_gray">
-    <color rgba="0.75 0.75 0.75 1.0"/>
+  <!-- Sensor boards (IMU, ToF) -->
+  <material name="blue">
+    <color rgba="0.0 0.25 0.8 1.0"/>
   </material>
-  <material name="silver">
-    <color rgba="0.82 0.82 0.82 1.0"/>
+  <!-- Camera module -->
+  <material name="camera_gray">
+    <color rgba="0.20 0.20 0.20 1.0"/>
   </material>
-  <material name="blue">
-    <color rgba="0.10 0.30 0.90 1.0"/>
+  <!-- Raspberry Pi board -->
+  <material name="green">
+    <color rgba="0.05 0.45 0.10 1.0"/>
   </material>
-  <material name="green">
-    <color rgba="0.10 0.80 0.20 1.0"/>
-  </material>
+  <!-- STM32 safety controller -->
   <material name="red">
-    <color rgba="0.90 0.10 0.10 1.0"/>
-  </material>
-  <material name="yellow">
-    <color rgba="1.00 0.90 0.10 1.0"/>
+    <color rgba="0.80 0.05 0.05 1.0"/>
   </material>
 </robot>
