Commit message: Create Gazebo simulation package

File: src/solarbot_description/urdf/common/properties.xacro (robot description, xacro)
@@ -1,44 +1,104 @@
 <?xml version="1.0"?>
 <robot xmlns:xacro="http://www.ros.org/wiki/xacro">
-  <!-- ========================================================= -->
-  <!-- CHASSIS DIMENSIONS (meters)                               -->
-  <!-- ========================================================= -->
-  <xacro:property name="chassis_length" value="0.393"/>
-  <xacro:property name="chassis_width"  value="0.206"/>
-  <xacro:property name="chassis_height" value="0.084"/>
-  <!-- ========================================================= -->
-  <!-- TRACK MODULES                                              -->
-  <!-- ========================================================= -->
-  <xacro:property name="track_length" value="0.115"/>
-  <xacro:property name="track_width"  value="0.050"/>
-  <xacro:property name="track_height" value="0.052"/>
-  <!-- Track module positions -->
-  <xacro:property name="front_track_x" value="0.125"/>
-  <xacro:property name="rear_track_x"  value="-0.125"/>
-  <xacro:property name="left_track_y"  value="0.128"/>
-  <xacro:property name="right_track_y" value="-0.128"/>
-  <!-- ========================================================= -->
-  <!-- ROBOT MASS                                                 -->
-  <!-- ========================================================= -->
-  <!-- Initial estimate -->
-  <xacro:property name="robot_mass" value="5.5"/>
-  <!-- ========================================================= -->
-  <!-- SENSOR POSITIONS                                           -->
-  <!-- ========================================================= -->
-  <!-- IMU -->
-  <xacro:property name="imu_x" value="0.0"/>
-  <xacro:property name="imu_y" value="0.0"/>
-  <xacro:property name="imu_z" value="0.020"/>
-  <!-- Downward Camera -->
-  <xacro:property name="camera_x" value="0.0"/>
-  <xacro:property name="camera_y" value="0.0"/>
-  <xacro:property name="camera_z" value="-0.030"/>
-  <!-- Forward ToF -->
-  <xacro:property name="front_tof_x" value="0.185"/>
-  <xacro:property name="front_tof_y" value="0.000"/>
-  <xacro:property name="front_tof_z" value="0.020"/>
-  <!-- Corner ToFs -->
-  <xacro:property name="corner_tof_x" value="0.160"/>
-  <xacro:property name="corner_tof_y" value="0.085"/>
-  <xacro:property name="corner_tof_z" value="-0.040"/>
+  <!--
+    properties.xacro
+    Single source of truth for ALL dimensions, masses and positions.
+    Edit numbers here — every other file picks them up automatically.
+    Real chassis measurements:
+      Total length : 393 mm
+      Total width  : 206 mm
+      Total height :  84 mm (tracks included)
+  -->
+  <!-- ── Chassis body ──────────────────────────────────────── -->
+  <xacro:property name="chassis_rail_length"  value="0.270"/>
+  <xacro:property name="chassis_rail_width"   value="0.055"/>
+  <xacro:property name="chassis_rail_height"  value="0.022"/>
+  <xacro:property name="plate_length"         value="0.105"/>
+  <xacro:property name="plate_width"          value="0.145"/>
+  <xacro:property name="plate_thickness"      value="0.008"/>
+  <xacro:property name="plate_z"              value="0.034"/>
+  <xacro:property name="side_rail_length"     value="0.295"/>
+  <xacro:property name="side_rail_width"      value="0.014"/>
+  <xacro:property name="side_rail_height"     value="0.018"/>
+  <xacro:property name="side_rail_z"          value="-0.006"/>
+  <xacro:property name="side_rail_y"          value="0.070"/>
+  <!-- ── Track geometry ───────────────────────────────────── -->
+  <xacro:property name="track_pod_length"     value="0.115"/>
+  <xacro:property name="track_pod_width"      value="0.050"/>
+  <xacro:property name="track_pod_height"     value="0.052"/>
+  <xacro:property name="track_full_length"    value="0.393"/>
+  <xacro:property name="track_front_x"        value="0.135"/>
+  <xacro:property name="track_rear_x"         value="-0.135"/>
+  <xacro:property name="track_y_offset"       value="0.078"/>
+  <xacro:property name="track_z_offset"       value="-0.016"/>
+  <!-- ── Virtual wheel (control) ──────────────────────────── -->
+  <xacro:property name="wheel_radius"         value="0.026"/>
+  <xacro:property name="wheel_width"          value="0.050"/>
+  <!-- ── Motors ───────────────────────────────────────────── -->
+  <xacro:property name="motor_radius"         value="0.018"/>
+  <xacro:property name="motor_shaft_length"   value="0.155"/>
+  <xacro:property name="motor_front_x"        value="0.155"/>
+  <xacro:property name="motor_z"              value="-0.006"/>
+  <!-- ── Base heights ─────────────────────────────────────── -->
+  <xacro:property name="base_z_above_ground"  value="${wheel_radius}"/>
+  <!-- ── Masses ────────────────────────────────────────────── -->
+  <xacro:property name="chassis_mass"         value="2.20"/>
+  <xacro:property name="track_pod_mass"       value="0.45"/>
+  <xacro:property name="virtual_wheel_mass"   value="0.001"/>
+  <!-- ══════════════════════════════════════════════════════ -->
+  <!-- ELECTRONICS POSITIONS                                 -->
+  <!-- All xyz relative to base_link origin.                 -->
+  <!-- Adjust once physical mounting is measured.            -->
+  <!-- ══════════════════════════════════════════════════════ -->
+  <!-- Battery pack (LiFePO4, centre-rear for balance) -->
+  <xacro:property name="battery_x"            value="-0.060"/>
+  <xacro:property name="battery_y"            value="0.000"/>
+  <xacro:property name="battery_z"            value="0.055"/>
+  <!-- Raspberry Pi 5 (rear top plate) -->
+  <xacro:property name="rpi_x"                value="-0.090"/>
+  <xacro:property name="rpi_y"                value="0.000"/>
+  <xacro:property name="rpi_z"                value="0.050"/>
+  <!-- ESP32 motor controller (front area, near motor driver) -->
+  <xacro:property name="esp32_x"              value="0.080"/>
+  <xacro:property name="esp32_y"              value="0.020"/>
+  <xacro:property name="esp32_z"              value="0.048"/>
+  <!-- STM32 safety controller (front top plate) -->
+  <xacro:property name="stm32_x"              value="0.080"/>
+  <xacro:property name="stm32_y"              value="-0.020"/>
+  <xacro:property name="stm32_z"              value="0.048"/>
+  <!-- ══════════════════════════════════════════════════════ -->
+  <!-- SENSOR POSITIONS                                      -->
+  <!-- All xyz relative to base_link origin.                 -->
+  <!-- ══════════════════════════════════════════════════════ -->
+  <!-- IMU (GY-91 / MPU9250 — centred on chassis) -->
+  <xacro:property name="imu_x"                value="0.000"/>
+  <xacro:property name="imu_y"                value="0.000"/>
+  <xacro:property name="imu_z"                value="0.045"/>
+  <!-- Downward camera (OV9732 — centre of chassis, looking down at panel) -->
+  <xacro:property name="camera_x"             value="0.000"/>
+  <xacro:property name="camera_y"             value="0.000"/>
+  <xacro:property name="camera_z"             value="-0.020"/>
+  <!-- Front obstacle ToF (forward-facing, above front edge) -->
+  <xacro:property name="front_tof_x"          value="0.200"/>
+  <xacro:property name="front_tof_y"          value="0.000"/>
+  <xacro:property name="front_tof_z"          value="0.010"/>
+  <!--
+    Corner cliff ToF sensors (downward-facing, detect panel edges).
+    Positioned just inboard of each track corner so they see the
+    panel surface drop-off before the wheels reach the edge.
+    rpy "0 0 0" = pointing straight down (sensor board faces -z).
+    Adjust x/y offsets once physically mounted and tested.
+  -->
+  <xacro:property name="front_left_tof_x"     value="0.170"/>
+  <xacro:property name="front_left_tof_y"     value="0.065"/>
+  <xacro:property name="front_left_tof_z"     value="-0.010"/>
+  <xacro:property name="front_right_tof_x"    value="0.170"/>
+  <xacro:property name="front_right_tof_y"    value="-0.065"/>
+  <xacro:property name="front_right_tof_z"    value="-0.010"/>
+  <xacro:property name="rear_left_tof_x"      value="-0.170"/>
+  <xacro:property name="rear_left_tof_y"      value="0.065"/>
+  <xacro:property name="rear_left_tof_z"      value="-0.010"/>
+  <xacro:property name="rear_right_tof_x"     value="-0.170"/>
+  <xacro:property name="rear_right_tof_y"     value="-0.065"/>
+  <xacro:property name="rear_right_tof_z"     value="-0.010"/>
 </robot>

File: src/solarbot_description/urdf/sensors/sensors.xacro (robot description, xacro)
@@ -1,4 +1,138 @@
 <?xml version="1.0"?>
 <robot xmlns:xacro="http://www.ros.org/wiki/xacro">
-    <!-- sensor definitions -->
+  <!--
+    sensors.xacro
+    ─────────────────────────────────────────────────────────────────
+    All sensor link and joint definitions.
+    Sensors:
+      imu_link                    GY-91 / MPU9250 IMU
+      downward_camera_link        OV9732 downward-facing camera
+      downward_camera_optical_frame  ROS optical frame (Z forward, X right)
+      front_tof_link              Forward obstacle ToF
+      front_left_tof_link  }
+      front_right_tof_link }      Corner cliff ToF sensors
+      rear_left_tof_link   }      (detect panel edges, face downward)
+      rear_right_tof_link  }
+    Published ROS topics (driver nodes, not defined here):
+      /imu
+      /camera/image_raw
+      /front_tof
+      /front_left_tof   /front_right_tof
+      /rear_left_tof    /rear_right_tof
+    All positions come from common/properties.xacro.
+    NOTE — camera optical frame rotation:
+      rpy="-1.5708 0 -1.5708" rotates the frame so that:
+        Z_optical points downward (-Z_base_link)
+        X_optical points forward  (+X_base_link)
+      This is the correct REP-103 camera optical convention for a
+      downward-facing camera.  Do NOT use "0 1.5708 0" — that
+      points the camera sideways.
+    Depends on: common/properties.xacro, common/materials.xacro
+  ─────────────────────────────────────────────────────────────────
+  -->
+  <!-- ── ToF sensor macro ──────────────────────────────────── -->
+  <!--
+    Reusable macro for any ToF sensor.
+    params:
+      name  — becomes ${name}_link and ${name}_joint
+      x y z — position relative to base_link
+      rpy   — orientation (e.g. "0 0 0" = downward, "0 1.5708 0" = forward)
+  -->
+  <xacro:macro name="tof_sensor" params="name x y z rpy">
+    <link name="${name}_link">
+      <visual>
+        <geometry>
+          <box size="0.025 0.025 0.015"/>
+        </geometry>
+        <material name="blue"/>
+      </visual>
+    </link>
+    <joint name="${name}_joint" type="fixed">
+      <parent link="base_link"/>
+      <child  link="${name}_link"/>
+      <origin xyz="${x} ${y} ${z}" rpy="${rpy}"/>
+    </joint>
+  </xacro:macro>
+  <!-- ── IMU ───────────────────────────────────────────────── -->
+  <link name="imu_link">
+    <visual>
+      <geometry>
+        <box size="0.025 0.025 0.008"/>
+      </geometry>
+      <material name="blue"/>
+    </visual>
+  </link>
+  <joint name="imu_joint" type="fixed">
+    <parent link="base_link"/>
+    <child  link="imu_link"/>
+    <origin xyz="${imu_x} ${imu_y} ${imu_z}" rpy="0 0 0"/>
+  </joint>
+  <!-- ── Downward camera ───────────────────────────────────── -->
+  <link name="downward_camera_link">
+    <visual>
+      <geometry>
+        <box size="0.030 0.030 0.020"/>
+      </geometry>
+      <material name="dark_gray"/>
+    </visual>
+  </link>
+  <joint name="downward_camera_joint" type="fixed">
+    <parent link="base_link"/>
+    <child  link="downward_camera_link"/>
+    <origin xyz="${camera_x} ${camera_y} ${camera_z}" rpy="0 0 0"/>
+  </joint>
+  <!--
+    Optical frame: massless, no visual.
+    The -1.5708 rotations convert from the ROS body convention
+    (X forward, Z up) to the camera optical convention
+    (Z forward = down into the panel, X right).
+  -->
+  <link name="downward_camera_optical_frame"/>
+  <joint name="downward_camera_optical_joint" type="fixed">
+    <parent link="downward_camera_link"/>
+    <child  link="downward_camera_optical_frame"/>
+    <origin xyz="0 0 -0.020" rpy="-1.5708 0 -1.5708"/>
+  </joint>
+  <!-- ── Front obstacle ToF (forward-facing) ───────────────── -->
+  <!--
+    rpy="0 1.5708 0" tilts the sensor to face forward (+X direction).
+    Detects obstacles ahead of the robot on the panel surface.
+  -->
+  <xacro:tof_sensor
+    name="front_tof"
+    x="${front_tof_x}"
+    y="${front_tof_y}"
+    z="${front_tof_z}"
+    rpy="0 1.5708 0"/>
+  <!-- ── Corner cliff ToF sensors (downward-facing) ────────── -->
+  <!--
+    rpy="0 0 0" — sensor faces straight down (-Z in base_link frame).
+    Placed at the four corners just inboard of the tracks so they
+    detect the panel edge drop-off before wheels reach it.
+    These feed edge_guard_node to trigger the safety stop + turn.
+  -->
+  <xacro:tof_sensor
+    name="front_left_tof"
+    x="${front_left_tof_x}"
+    y="${front_left_tof_y}"
+    z="${front_left_tof_z}"
+    rpy="0 0 0"/>
+  <xacro:tof_sensor
+    name="front_right_tof"
+    x="${front_right_tof_x}"
+    y="${front_right_tof_y}"
+    z="${front_right_tof_z}"
+    rpy="0 0 0"/>
+  <xacro:tof_sensor
+    name="rear_left_tof"
+    x="${rear_left_tof_x}"
+    y="${rear_left_tof_y}"
+    z="${rear_left_tof_z}"
+    rpy="0 0 0"/>
+  <xacro:tof_sensor
+    name="rear_right_tof"
+    x="${rear_right_tof_x}"
+    y="${rear_right_tof_y}"
+    z="${rear_right_tof_z}"
+    rpy="0 0 0"/>
 </robot>

File: src/solarbot_description/urdf/solarbot.urdf.xacro (robot description, xacro)
@@ -1,18 +1,32 @@
 <?xml version="1.0"?>
-<robot name="solarbot"
-       xmlns:xacro="http://www.ros.org/wiki/xacro">
-  <!-- ===================================================== -->
-  <!-- Common -->
-  <!-- ===================================================== -->
+<robot name="solarbot" xmlns:xacro="http://www.ros.org/wiki/xacro">
+  <!--
+    solarbot.urdf.xacro
+    ─────────────────────────────────────────────────────────────────
+    Top-level robot description.  This file only includes sub-files —
+    no geometry, no joints, no properties are defined here.
+    Include order matters:
+      1. common/  — properties and materials must come first because
+                    every other file references their xacro:property values
+      2. base/    — structural links and joints
+      3. sensors/ — sensor frames (depends on base links existing)
+      4. electronics/ — board visuals (depends on base links existing)
+      5. control/ — ros2_control block (references joint names from base/)
+    Launch args forwarded to sub-files:
+      use_real_hardware  (default: false)  — selects hardware plugin
+      serial_port        (default: /dev/ttyACM0)
+  ─────────────────────────────────────────────────────────────────
+  -->
+  <!-- ── 1. Common: properties and materials ─────────────────── -->
   <xacro:include filename="$(find solarbot_description)/urdf/common/properties.xacro"/>
   <xacro:include filename="$(find solarbot_description)/urdf/common/materials.xacro"/>
-  <!-- ===================================================== -->
-  <!-- Base -->
-  <!-- ===================================================== -->
+  <!-- ── 2. Base: chassis body and tracks ────────────────────── -->
   <xacro:include filename="$(find solarbot_description)/urdf/base/chassis.xacro"/>
   <xacro:include filename="$(find solarbot_description)/urdf/base/tracks.xacro"/>
-  <!-- ===================================================== -->
-  <!-- Sensors -->
-  <!-- ===================================================== -->
+  <!-- ── 3. Sensors ───────────────────────────────────────────── -->
   <xacro:include filename="$(find solarbot_description)/urdf/sensors/sensors.xacro"/>
+  <!-- ── 4. Electronics ───────────────────────────────────────── -->
+  <xacro:include filename="$(find solarbot_description)/urdf/electronics/electronics.xacro"/>
+  <!-- ── 5. ros2_control ──────────────────────────────────────── -->
+  <xacro:include filename="$(find solarbot_description)/urdf/control/ros2_control.xacro"/>
 </robot>
