Commit message: urdf updated

File: src/solarbot_description/urdf/base/chassis.xacro (robot description, xacro)
@@ -2,53 +2,23 @@
 <robot xmlns:xacro="http://www.ros.org/wiki/xacro">
   <!--
-    chassis.xacro
-    ─────────────────────────────────────────────────────────────────
-    Main chassis body: base_footprint, base_link.
-    Visuals represent the aluminium frame as seen on the real chassis:
-      • Central spine rail
-      • Front and rear top mounting plates
-      • Left and right side rails
-    Depends on: common/properties.xacro, common/materials.xacro
-  ─────────────────────────────────────────────────────────────────
+    chassis.xacro  —  base_footprint + base_link frame only.
+    Track pods moved back to tracks.xacro (they are now real physics
+    objects). Motor shaft visuals remain inline here since they are
+    purely cosmetic with no physics role.
   -->
-  <!-- ── Inertia helper macros ─────────────────────────────── -->
-  <!-- Solid box: m=mass, lx/ly/lz=dimensions along each axis -->
   <xacro:macro name="box_inertia" params="m lx ly lz">
     <inertia
-      ixx="${m*(ly*ly + lz*lz)/12.0}"
-      ixy="0.0" ixz="0.0"
-      iyy="${m*(lx*lx + lz*lz)/12.0}"
-      iyz="0.0"
+      ixx="${m*(ly*ly + lz*lz)/12.0}" ixy="0" ixz="0"
+      iyy="${m*(lx*lx + lz*lz)/12.0}" iyz="0"
       izz="${m*(lx*lx + ly*ly)/12.0}"/>
   </xacro:macro>
-  <!-- Solid cylinder: m=mass, r=radius, h=height along spin axis -->
-  <xacro:macro name="cylinder_inertia" params="m r h">
-    <inertia
-      ixx="${m*(3.0*r*r + h*h)/12.0}"
-      ixy="0.0" ixz="0.0"
-      iyy="${m*(3.0*r*r + h*h)/12.0}"
-      iyz="0.0"
-      izz="${m*r*r/2.0}"/>
-  </xacro:macro>
-  <!-- ── base_footprint ────────────────────────────────────── -->
-  <!--
-    Projection of the robot onto the ground plane.
-    Nav2 and the localisation stack use this frame as the
-    reference for 2D pose (x, y, yaw).
-  -->
+  <!-- base_footprint — ground-plane projection, used by Nav2 -->
   <link name="base_footprint"/>
   <joint name="base_footprint_joint" type="fixed">
     <parent link="base_footprint"/>
     <child  link="base_link"/>
-    <!-- Raise base_link so the track bottoms sit at z=0 in the world -->
     <origin xyz="0 0 ${base_z_above_ground}" rpy="0 0 0"/>
   </joint>
-  <!-- ── base_link ─────────────────────────────────────────── -->
-  <!--
-    Rigid chassis body.  The inertial block approximates the full
-    chassis as a solid box — good enough for simulation dynamics.
-    Visuals are broken into sub-boxes to resemble the real aluminium
-    frame visible in the chassis photo.
-  -->
+  <!-- base_link — rigid chassis body -->
   <link name="base_link">
     <inertial>
@@ -61,11 +31,9 @@
         lz="${track_pod_height}"/>
     </inertial>
-    <!-- ── Visual: central spine rail ── -->
+    <!-- Central spine rail -->
     <visual>
       <origin xyz="0 0 0" rpy="0 0 0"/>
       <geometry>
-        <box size="${chassis_rail_length}
-                   ${chassis_rail_width}
-                   ${chassis_rail_height}"/>
+        <box size="${chassis_rail_length} ${chassis_rail_width} ${chassis_rail_height}"/>
       </geometry>
       <material name="silver"/>
@@ -74,16 +42,12 @@
       <origin xyz="0 0 0" rpy="0 0 0"/>
       <geometry>
-        <box size="${chassis_rail_length}
-                   ${chassis_rail_width}
-                   ${chassis_rail_height}"/>
+        <box size="${chassis_rail_length} ${chassis_rail_width} ${chassis_rail_height}"/>
       </geometry>
     </collision>
-    <!-- ── Visual: front top plate ── -->
+    <!-- Front top plate -->
     <visual>
       <origin xyz="${plate_length} 0 ${plate_z}" rpy="0 0 0"/>
       <geometry>
-        <box size="${plate_length}
-                   ${plate_width}
-                   ${plate_thickness}"/>
+        <box size="${plate_length} ${plate_width} ${plate_thickness}"/>
       </geometry>
       <material name="silver"/>
@@ -92,16 +56,12 @@
       <origin xyz="${plate_length} 0 ${plate_z}" rpy="0 0 0"/>
       <geometry>
-        <box size="${plate_length}
-                   ${plate_width}
-                   ${plate_thickness}"/>
+        <box size="${plate_length} ${plate_width} ${plate_thickness}"/>
       </geometry>
     </collision>
-    <!-- ── Visual: rear top plate ── -->
+    <!-- Rear top plate -->
     <visual>
       <origin xyz="${-plate_length} 0 ${plate_z}" rpy="0 0 0"/>
       <geometry>
-        <box size="${plate_length}
-                   ${plate_width}
-                   ${plate_thickness}"/>
+        <box size="${plate_length} ${plate_width} ${plate_thickness}"/>
       </geometry>
       <material name="silver"/>
@@ -110,26 +70,36 @@
       <origin xyz="${-plate_length} 0 ${plate_z}" rpy="0 0 0"/>
       <geometry>
-        <box size="${plate_length}
-                   ${plate_width}
-                   ${plate_thickness}"/>
+        <box size="${plate_length} ${plate_width} ${plate_thickness}"/>
       </geometry>
     </collision>
-    <!-- ── Visual: left side rail ── -->
+    <!-- Left side rail (visual only) -->
     <visual>
       <origin xyz="0 ${side_rail_y} ${side_rail_z}" rpy="0 0 0"/>
       <geometry>
-        <box size="${side_rail_length}
-                   ${side_rail_width}
-                   ${side_rail_height}"/>
+        <box size="${side_rail_length} ${side_rail_width} ${side_rail_height}"/>
       </geometry>
       <material name="silver"/>
     </visual>
-    <!-- ── Visual: right side rail ── -->
+    <!-- Right side rail (visual only) -->
     <visual>
       <origin xyz="0 ${-side_rail_y} ${side_rail_z}" rpy="0 0 0"/>
       <geometry>
-        <box size="${side_rail_length}
-                   ${side_rail_width}
-                   ${side_rail_height}"/>
+        <box size="${side_rail_length} ${side_rail_width} ${side_rail_height}"/>
+      </geometry>
+      <material name="silver"/>
+    </visual>
+    <!-- Front motor shaft (visual only) -->
+    <visual>
+      <origin xyz="${motor_front_x} 0 ${motor_z}" rpy="1.5708 0 0"/>
+      <geometry>
+        <cylinder radius="${motor_radius}" length="${motor_shaft_length}"/>
+      </geometry>
+      <material name="silver"/>
+    </visual>
+    <!-- Rear motor shaft (visual only) -->
+    <visual>
+      <origin xyz="${-motor_front_x} 0 ${motor_z}" rpy="1.5708 0 0"/>
+      <geometry>
+        <cylinder radius="${motor_radius}" length="${motor_shaft_length}"/>
       </geometry>
       <material name="silver"/>

File: src/solarbot_description/urdf/base/tracks.xacro (robot description, xacro)
@@ -4,143 +4,97 @@
     tracks.xacro
     ─────────────────────────────────────────────────────────────────
-    Track pods (4 × fixed visual boxes), motor shaft visuals (2),
-    and virtual wheel joints (2) for diff_drive_controller.
-    Why virtual wheels?
-      diff_drive_controller requires continuous revolute joints to
-      send velocity commands to.  The 4 track pod joints are fixed
-      (they are rigid visual elements — tracks don't steer or pivot).
-      We therefore add two invisible virtual wheel links — one at
-      the lateral centre of each track side — that the controller
-      can command.  The Arduino firmware then mirrors each side's
-      command to both physical motors on that side.
-    Joint names used here MUST match diff_drive_controller config:
-      left_wheel_joint   ← left track
-      right_wheel_joint  ← right track
+    Four track pod links — each is a real physics object.
+    No virtual wheel links. Each track pod IS the wheel:
+        ┌──────────────────┐   ← box VISUAL  (track appearance)
+        │                  │
+        │      ╔════╗      │   ← cylinder COLLISION  (rolls on ground)
+        │      ║ O  ║      │     radius = wheel_radius = 0.026 m
+        │      ╚════╝      │     length = track_pod_width  = 0.050 m
+        │                  │
+        └──────────────────┘
+    Why cylinder collision, box visual?
+      • The cylinder is what Gazebo's ODE solver rolls on the ground —
+        it produces a clean, stable single contact line per pod.
+      • The box visual is the appearance of the rubber track.
+      • A box collision would have 4 contact points that fight each
+        other and make the robot jitter.
+    DiffDrive drives all 4 joints as two pairs:
+      LEFT  pair: front_left_wheel_joint + rear_left_wheel_joint
+      RIGHT pair: front_right_wheel_joint + rear_right_wheel_joint
+    Joint naming convention: ${name}_wheel_joint
+      This is what gazebo.xacro DiffDrive plugin and
+      ros2_control.xacro both reference.
     Depends on: common/properties.xacro, common/materials.xacro
   ─────────────────────────────────────────────────────────────────
   -->
+  <xacro:macro name="cylinder_inertia" params="m r h">
+    <inertia
+      ixx="${m*(3.0*r*r + h*h)/12.0}" ixy="0" ixz="0"
+      iyy="${m*(3.0*r*r + h*h)/12.0}" iyz="0"
+      izz="${m*r*r/2.0}"/>
+  </xacro:macro>
   <!-- ══════════════════════════════════════════════════════════ -->
-  <!-- Macro: single track pod (box visual, fixed joint)        -->
+  <!-- track_pod macro                                           -->
   <!-- ══════════════════════════════════════════════════════════ -->
   <xacro:macro name="track_pod" params="name x y">
     <link name="${name}_track_link">
+      <!--
+        Inertia: modelled as a solid cylinder (not box) to match the
+        cylinder collision shape. mass = 0.45 kg per pod.
+      -->
       <inertial>
         <origin xyz="0 0 0" rpy="0 0 0"/>
         <mass value="${track_pod_mass}"/>
-        <inertia
-          ixx="${track_pod_mass*(track_pod_width*track_pod_width  + track_pod_height*track_pod_height)/12.0}"
-          ixy="0" ixz="0"
-          iyy="${track_pod_mass*(track_pod_length*track_pod_length + track_pod_height*track_pod_height)/12.0}"
-          iyz="0"
-          izz="${track_pod_mass*(track_pod_length*track_pod_length + track_pod_width*track_pod_width)/12.0}"/>
+        <xacro:cylinder_inertia
+          m="${track_pod_mass}"
+          r="${wheel_radius}"
+          h="${track_pod_width}"/>
       </inertial>
+      <!-- VISUAL: box → the rubber track appearance -->
       <visual>
         <origin xyz="0 0 0" rpy="0 0 0"/>
         <geometry>
-          <box size="${track_pod_length}
-                     ${track_pod_width}
-                     ${track_pod_height}"/>
+          <box size="${track_pod_length} ${track_pod_width} ${track_pod_height}"/>
         </geometry>
         <material name="black"/>
       </visual>
+      <!--
+        COLLISION: cylinder → the rolling contact surface.
+        rpy="1.5708 0 0" rotates the cylinder from its default
+        z-axis orientation to the y-axis so it rolls when the
+        joint spins around y (axis xyz="0 1 0" in the joint below).
+        Radius = wheel_radius = 0.026 m.
+        The joint origin places the cylinder centre exactly at
+        ground contact height.
+      -->
       <collision>
-        <origin xyz="0 0 0" rpy="0 0 0"/>
+        <origin xyz="0 0 0" rpy="1.5708 0 0"/>
         <geometry>
-          <box size="${track_pod_length}
-                     ${track_pod_width}
-                     ${track_pod_height}"/>
+          <cylinder radius="${wheel_radius}" length="${track_pod_width}"/>
         </geometry>
       </collision>
     </link>
-    <!-- Fixed joint: track pod is rigidly attached to chassis -->
-    <joint name="${name}_track_joint" type="fixed">
+    <!--
+      Continuous joint — DiffDrive can command velocity on this.
+      Joint origin z = -wheel_radius from base_link.
+      base_link is at z = wheel_radius above ground (base_z_above_ground).
+      Therefore wheel centre in world frame = wheel_radius - wheel_radius = 0,
+      i.e. at ground level. Gazebo contact dynamics with minDepth handle
+      the small cylinder–ground overlap.
+    -->
+    <joint name="${name}_wheel_joint" type="continuous">
       <parent link="base_link"/>
       <child  link="${name}_track_link"/>
-      <origin xyz="${x} ${y} ${track_z_offset}" rpy="0 0 0"/>
+      <origin xyz="${x} ${y} ${-wheel_radius}" rpy="0 0 0"/>
+      <axis xyz="0 1 0"/>
+      <dynamics damping="0.05" friction="0.1"/>
     </joint>
   </xacro:macro>
   <!-- ══════════════════════════════════════════════════════════ -->
-  <!-- Macro: virtual wheel link + continuous joint              -->
+  <!-- Instantiate all four track pods                          -->
   <!-- ══════════════════════════════════════════════════════════ -->
-  <xacro:macro name="virtual_wheel" params="name y_offset">
-    <!--
-      No visual or collision — purely a control artifact.
-      Placed at the lateral centre of each track at ground-contact
-      height (z = -wheel_radius from base_link = ground level).
-    -->
-    <link name="${name}_virtual_wheel_link">
-      <inertial>
-        <origin xyz="0 0 0" rpy="0 0 0"/>
-        <mass value="${virtual_wheel_mass}"/>
-        <inertia
-          ixx="${virtual_wheel_mass*(3.0*wheel_radius*wheel_radius + wheel_width*wheel_width)/12.0}"
-          ixy="0" ixz="0"
-          iyy="${virtual_wheel_mass*(3.0*wheel_radius*wheel_radius + wheel_width*wheel_width)/12.0}"
-          iyz="0"
-          izz="${virtual_wheel_mass*wheel_radius*wheel_radius/2.0}"/>
-      </inertial>
-    </link>
-    <joint name="${name}_wheel_joint" type="continuous">
-      <parent link="base_link"/>
-      <child  link="${name}_virtual_wheel_link"/>
-      <!-- Centred longitudinally (x=0), at track y, at contact height -->
-      <origin xyz="0 ${y_offset} ${-wheel_radius}" rpy="0 0 0"/>
-      <!-- Standard diff-drive: wheel spins around the lateral (y) axis -->
-      <axis xyz="0 1 0"/>
-      <dynamics damping="0.01" friction="0.1"/>
-    </joint>
-  </xacro:macro>
-  <!-- ══════════════════════════════════════════════════════════ -->
-  <!-- Instantiate four track pods                              -->
-  <!-- ══════════════════════════════════════════════════════════ -->
-  <xacro:track_pod name="front_left"
-                   x="${track_front_x}"
-                   y="${track_y_offset}"/>
-  <xacro:track_pod name="rear_left"
-                   x="${track_rear_x}"
-                   y="${track_y_offset}"/>
-  <xacro:track_pod name="front_right"
-                   x="${track_front_x}"
-                   y="${-track_y_offset}"/>
-  <xacro:track_pod name="rear_right"
-                   x="${track_rear_x}"
-                   y="${-track_y_offset}"/>
-  <!-- ══════════════════════════════════════════════════════════ -->
-  <!-- Motor shaft visuals (fixed, cosmetic only)               -->
-  <!-- ══════════════════════════════════════════════════════════ -->
-  <link name="front_motor_link">
-    <visual>
-      <!-- rpy rotates the cylinder to lie along the y-axis (lateral) -->
-      <origin xyz="0 0 0" rpy="1.5708 0 0"/>
-      <geometry>
-        <cylinder radius="${motor_radius}" length="${motor_shaft_length}"/>
-      </geometry>
-      <material name="silver"/>
-    </visual>
-  </link>
-  <joint name="front_motor_joint" type="fixed">
-    <parent link="base_link"/>
-    <child  link="front_motor_link"/>
-    <origin xyz="${motor_front_x} 0 ${motor_z}" rpy="0 0 0"/>
-  </joint>
-  <link name="rear_motor_link">
-    <visual>
-      <origin xyz="0 0 0" rpy="1.5708 0 0"/>
-      <geometry>
-        <cylinder radius="${motor_radius}" length="${motor_shaft_length}"/>
-      </geometry>
-      <material name="silver"/>
-    </visual>
-  </link>
-  <joint name="rear_motor_joint" type="fixed">
-    <parent link="base_link"/>
-    <child  link="rear_motor_link"/>
-    <origin xyz="${-motor_front_x} 0 ${motor_z}" rpy="0 0 0"/>
-  </joint>
-  <!-- ══════════════════════════════════════════════════════════ -->
-  <!-- Two virtual wheel joints (one per track side)            -->
-  <!-- These are what diff_drive_controller actually commands.  -->
-  <!-- ══════════════════════════════════════════════════════════ -->
-  <xacro:virtual_wheel name="left"  y_offset="${track_y_offset}"/>
-  <xacro:virtual_wheel name="right" y_offset="${-track_y_offset}"/>
+  <xacro:track_pod name="front_left"  x="${track_front_x}" y="${track_y_offset}"/>
+  <xacro:track_pod name="rear_left"   x="${track_rear_x}"  y="${track_y_offset}"/>
+  <xacro:track_pod name="front_right" x="${track_front_x}" y="${-track_y_offset}"/>
+  <xacro:track_pod name="rear_right"  x="${track_rear_x}"  y="${-track_y_offset}"/>
 </robot>

File: src/solarbot_description/urdf/control/ros2_control.xacro (robot description, xacro)
@@ -1,65 +1,46 @@
 <?xml version="1.0"?>
 <robot xmlns:xacro="http://www.ros.org/wiki/xacro">
-  <!-- ==========================================================
-       ROS2 Control Configuration
-       ========================================================== -->
+  <!--
+    ros2_control.xacro
+    Updated to reference all 4 track wheel joints (front + rear per side).
+    On real hardware these are electrically paired (L+L, R+R) so commanding
+    both joints on each side with the same value is physically correct.
+  -->
   <xacro:arg name="use_real_hardware" default="false"/>
-  <xacro:arg name="serial_port" default="/dev/ttyACM0"/>
-  <xacro:arg name="baud_rate" default="115200"/>
-  <ros2_control name="SolarbotSystem" type="system">
-    <!-- ===================================================== -->
-    <!-- Hardware Plugin                                       -->
-    <!-- ===================================================== -->
+  <xacro:arg name="serial_port"       default="/dev/ttyACM0"/>
+  <ros2_control name="SolarbotHardware" type="system">
     <hardware>
-      <!-- Simulation -->
-      <xacro:unless value="$(arg use_real_hardware)">
-        <plugin>gz_ros2_control/GazeboSimSystem</plugin>
-      </xacro:unless>
-      <!-- Real Robot -->
       <xacro:if value="$(arg use_real_hardware)">
         <plugin>panelbot_hardware/SkidSteerHardware</plugin>
-        <param name="serial_port">
-          $(arg serial_port)
-        </param>
-        <param name="baud_rate">
-          $(arg baud_rate)
-        </param>
-        <param name="wheel_radius">
-          ${wheel_radius}
-        </param>
-        <param name="wheel_separation">
-          ${2.0 * track_y_offset}
-        </param>
-        <param name="max_wheel_rad_s">
-          6.0
-        </param>
+        <param name="serial_port">$(arg serial_port)</param>
+        <param name="baud_rate">115200</param>
+        <param name="wheel_radius">${wheel_radius}</param>
+        <param name="max_wheel_rad_s">6.0</param>
       </xacro:if>
+      <xacro:unless value="$(arg use_real_hardware)">
+        <plugin>mock_components/GenericSystem</plugin>
+        <param name="calculate_dynamics">true</param>
+      </xacro:unless>
     </hardware>
-    <!-- ===================================================== -->
-    <!-- Left Drive Joint                                      -->
-    <!-- ===================================================== -->
-    <joint name="left_wheel_joint">
+    <joint name="front_left_wheel_joint">
       <command_interface name="velocity"/>
-      <state_interface name="position"/>
-      <state_interface name="velocity"/>
+      <state_interface   name="velocity"/>
+      <state_interface   name="position"/>
     </joint>
-    <!-- ===================================================== -->
-    <!-- Right Drive Joint                                     -->
-    <!-- ===================================================== -->
-    <joint name="right_wheel_joint">
+    <joint name="rear_left_wheel_joint">
       <command_interface name="velocity"/>
-      <state_interface name="position"/>
-      <state_interface name="velocity"/>
+      <state_interface   name="velocity"/>
+      <state_interface   name="position"/>
+    </joint>
+    <joint name="front_right_wheel_joint">
+      <command_interface name="velocity"/>
+      <state_interface   name="velocity"/>
+      <state_interface   name="position"/>
+    </joint>
+    <joint name="rear_right_wheel_joint">
+      <command_interface name="velocity"/>
+      <state_interface   name="velocity"/>
+      <state_interface   name="position"/>
     </joint>
   </ros2_control>
-  <!-- ==========================================================
-       Gazebo Plugin
-       ========================================================== -->
-  <gazebo>
-    <plugin
-      filename="gz_ros2_control-system"
-      name="gz_ros2_control::GazeboSimROS2ControlPlugin">
-      <parameters>$(find solarbot_description)/config/controllers.yaml</parameters>
-    </plugin>
-  </gazebo>
 </robot>
