Commit message: urdf updated

File: src/solarbot_description/urdf/gazebo/gazebo.xacro (robot description, xacro)
@@ -2,45 +2,43 @@
 <robot xmlns:xacro="http://www.ros.org/wiki/xacro">
   <!--
-    gazebo.xacro
-    ─────────────────────────────────────────────────────────────────
-    Gazebo Harmonic (gz-sim) plugin and sensor definitions.
-    This file is ONLY relevant when running in simulation.
-    It has no effect on real-hardware launches.
-    Contents:
-      1. gz_ros2_control plugin  — connects ros2_control controllers
-                                   to Gazebo joint physics
-      2. IMU sensor              — publishes /imu
-      3. Downward camera         — publishes /camera/image_raw
-      4. Cliff ToF sensors × 4  — /front_left_tof etc. (edge detection)
-      5. Front obstacle ToF      — /front_tof (forward range)
-      6. Gazebo material colours — so links render correctly in Gazebo
-                                   (Gazebo ignores URDF <material> tags)
-    Topic names here MUST match the ros_gz_bridge entries in gazebo.launch.py.
-    Depends on: common/properties.xacro (for wheel_radius, sensor positions)
-  ─────────────────────────────────────────────────────────────────
+    gazebo.xacro — Gazebo Harmonic plugin and sensor definitions.
+    Updated: DiffDrive drives all 4 track joints, friction on all 4 pods.
   -->
-  <!-- ══════════════════════════════════════════════════════════ -->
-  <!-- 1. gz_ros2_control plugin                                 -->
-  <!-- ══════════════════════════════════════════════════════════ -->
-  <!--
-    This is the Gazebo Harmonic equivalent of the old
-    libgazebo_ros2_control.so plugin.  It reads the <ros2_control>
-    block from the URDF, loads the hardware plugin declared there
-    (mock_components/GenericSystem for simulation), and connects
-    it to Gazebo's joint state/command interface so that
-    diff_drive_controller actually moves the simulated robot.
-    The parameters file path tells it where to find controllers.yaml.
-    This must match the path passed to the controller spawner in
-    gazebo.launch.py.
-  -->
-  <!-- ══════════════════════════════════════════════════════════ -->
-  <!-- 2. IMU sensor (GY-91 / MPU9250)                          -->
-  <!-- ══════════════════════════════════════════════════════════ -->
-  <!--
-    Attached to imu_link (defined in sensors/sensors.xacro).
-    Noise values approximate MPU9250 datasheet figures.
-    update_rate: 100 Hz matches real sensor capability.
-    Topic: /imu  →  bridged to ROS2 by ros_gz_bridge.
-  -->
+  <!-- ══ 1. DiffDrive plugin (replaces gz_ros2_control) ══════ -->
+  <gazebo>
+    <plugin filename="gz-sim-diff-drive-system"
+            name="gz::sim::systems::DiffDrive">
+      <!-- LEFT pair -->
+      <left_joint>front_left_wheel_joint</left_joint>
+      <left_joint>rear_left_wheel_joint</left_joint>
+      <!-- RIGHT pair -->
+      <right_joint>front_right_wheel_joint</right_joint>
+      <right_joint>rear_right_wheel_joint</right_joint>
+      <wheel_separation>0.156</wheel_separation>
+      <wheel_radius>0.026</wheel_radius>
+      <odom_publish_frequency>30</odom_publish_frequency>
+      <topic>cmd_vel</topic>
+      <odom_topic>odometry</odom_topic>
+      <tf_topic>tf</tf_topic>
+      <frame_id>odom</frame_id>
+      <child_frame_id>base_footprint</child_frame_id>
+      <max_linear_acceleration>0.5</max_linear_acceleration>
+      <max_angular_acceleration>1.0</max_angular_acceleration>
+      <min_velocity>-0.15</min_velocity>
+      <max_velocity>0.15</max_velocity>
+    </plugin>
+  </gazebo>
+  <!-- Joint state publisher — publishes all 4 wheel joint states -->
+  <gazebo>
+    <plugin filename="gz-sim-joint-state-publisher-system"
+            name="gz::sim::systems::JointStatePublisher">
+      <joint_name>front_left_wheel_joint</joint_name>
+      <joint_name>rear_left_wheel_joint</joint_name>
+      <joint_name>front_right_wheel_joint</joint_name>
+      <joint_name>rear_right_wheel_joint</joint_name>
+      <topic>joint_states</topic>
+    </plugin>
+  </gazebo>
+  <!-- ══ 2. IMU sensor ════════════════════════════════════════ -->
   <gazebo reference="imu_link">
     <sensor name="imu_sensor" type="imu">
@@ -63,20 +61,5 @@
     </sensor>
   </gazebo>
-  <!-- ══════════════════════════════════════════════════════════ -->
-  <!-- 3. Downward camera (OV9732, 720p)                        -->
-  <!-- ══════════════════════════════════════════════════════════ -->
-  <!--
-    Mounted under the chassis (downward_camera_link, defined in
-    sensors/sensors.xacro).  Looking straight down at the panel surface.
-    FOV: 78° horizontal (OV9732 spec, wide enough to see panel texture).
-    Resolution: 640×480 — sufficient for ECC visual odometry without
-    overloading the Pi's CPU.
-    Near clip: 0.01 m — camera is ~6 mm above panel surface, so keep
-    near clip well below that.
-    Far clip: 0.5 m — only need to see the panel surface below.
-    Topics (bridged via ros_gz_bridge):
-      /camera/image_raw       sensor_msgs/Image
-      /camera/camera_info     sensor_msgs/CameraInfo
-  -->
+  <!-- ══ 3. Downward camera ═══════════════════════════════════ -->
   <gazebo reference="downward_camera_link">
     <sensor name="downward_camera" type="camera">
@@ -86,5 +69,4 @@
       <gz_frame_id>downward_camera_optical_frame</gz_frame_id>
       <camera name="downward_camera">
-        <!-- OV9732: 78° HFOV -->
         <horizontal_fov>1.3614</horizontal_fov>
         <image>
@@ -102,32 +84,8 @@
           <stddev>0.005</stddev>
         </noise>
-        <distortion>
-          <k1>0.0</k1>
-          <k2>0.0</k2>
-          <k3>0.0</k3>
-          <p1>0.0</p1>
-          <p2>0.0</p2>
-        </distortion>
       </camera>
     </sensor>
   </gazebo>
-  <!-- ══════════════════════════════════════════════════════════ -->
-  <!-- 4. Cliff ToF sensors (downward, edge detection)          -->
-  <!-- ══════════════════════════════════════════════════════════ -->
-  <!--
-    Modelled as single-beam GPU lidars (best ToF approximation in
-    Gazebo Harmonic).  Each sensor fires a narrow beam straight down
-    (-z in sensor frame, which is -z in base_link for these sensors).
-    Range spec (approximates VL53L0X / VL53L1X):
-      min: 0.01 m   max: 1.20 m   resolution: 0.001 m
-    When the robot is on a panel (z=0.04) and the sensor is at
-    z=-0.010 from base_link (base_link at z=0.066 from ground):
-      expected reading = 0.066 - 0.010 - 0.040 = 0.016 m (on panel)
-    When the robot reaches a panel edge (gap, z=0):
-      expected reading = 0.066 - 0.010 - 0.000 = 0.056 m (deeper)
-    edge_guard_node threshold sits between these two values.
-    Topics bridged: /front_left_tof, /front_right_tof,
-                    /rear_left_tof,  /rear_right_tof
-  -->
+  <!-- ══ 4. Cliff ToF macro (single-beam lidar) ══════════════ -->
   <xacro:macro name="cliff_tof_gazebo" params="link_name topic">
     <gazebo reference="${link_name}">
@@ -139,27 +97,18 @@
         <lidar>
           <scan>
-            <!-- Single beam: 1 horizontal × 1 vertical ray -->
             <horizontal>
-              <samples>1</samples>
-              <resolution>1</resolution>
-              <min_angle>0</min_angle>
-              <max_angle>0</max_angle>
+              <samples>1</samples><resolution>1</resolution>
+              <min_angle>0</min_angle><max_angle>0</max_angle>
             </horizontal>
             <vertical>
-              <samples>1</samples>
-              <resolution>1</resolution>
-              <min_angle>0</min_angle>
-              <max_angle>0</max_angle>
+              <samples>1</samples><resolution>1</resolution>
+              <min_angle>0</min_angle><max_angle>0</max_angle>
             </vertical>
           </scan>
           <range>
-            <min>0.010</min>
-            <max>1.200</max>
-            <resolution>0.001</resolution>
+            <min>0.010</min><max>1.200</max><resolution>0.001</resolution>
           </range>
           <noise>
-            <type>gaussian</type>
-            <mean>0.0</mean>
-            <stddev>0.002</stddev>
+            <type>gaussian</type><mean>0.0</mean><stddev>0.002</stddev>
           </noise>
         </lidar>
@@ -171,13 +120,5 @@
   <xacro:cliff_tof_gazebo link_name="rear_left_tof_link"   topic="/rear_left_tof"/>
   <xacro:cliff_tof_gazebo link_name="rear_right_tof_link"  topic="/rear_right_tof"/>
-  <!-- ══════════════════════════════════════════════════════════ -->
-  <!-- 5. Front obstacle ToF (forward-facing)                   -->
-  <!-- ══════════════════════════════════════════════════════════ -->
-  <!--
-    Faces +x (forward).  Same single-beam lidar approach.
-    Used by drive_node / safety layer to detect obstacles ahead
-    on the panel surface (e.g. panel frame lip, foreign object).
-    Topic: /front_tof
-  -->
+  <!-- ══ 5. Front obstacle ToF ════════════════════════════════ -->
   <gazebo reference="front_tof_link">
     <sensor name="front_tof_sensor" type="gpu_lidar">
@@ -189,99 +130,59 @@
         <scan>
           <horizontal>
-            <samples>1</samples>
-            <resolution>1</resolution>
-            <min_angle>0</min_angle>
-            <max_angle>0</max_angle>
+            <samples>1</samples><resolution>1</resolution>
+            <min_angle>0</min_angle><max_angle>0</max_angle>
           </horizontal>
           <vertical>
-            <samples>1</samples>
-            <resolution>1</resolution>
-            <min_angle>0</min_angle>
-            <max_angle>0</max_angle>
+            <samples>1</samples><resolution>1</resolution>
+            <min_angle>0</min_angle><max_angle>0</max_angle>
           </vertical>
         </scan>
         <range>
-          <min>0.010</min>
-          <max>2.000</max>
-          <resolution>0.001</resolution>
+          <min>0.010</min><max>2.000</max><resolution>0.001</resolution>
         </range>
         <noise>
-          <type>gaussian</type>
-          <mean>0.0</mean>
-          <stddev>0.003</stddev>
+          <type>gaussian</type><mean>0.0</mean><stddev>0.003</stddev>
         </noise>
       </lidar>
     </sensor>
   </gazebo>
-  <!-- ══════════════════════════════════════════════════════════ -->
-  <!-- 6. Gazebo material colours                                -->
-  <!-- ══════════════════════════════════════════════════════════ -->
+  <!-- ══ 6. Track pod friction (all four pods) ════════════════ -->
   <!--
-    Gazebo Harmonic ignores the <material> tags inside URDF <visual>
-    elements.  These <gazebo reference="..."> blocks set the actual
-    rendered colours in Gazebo.
-    Omitting these makes everything grey in the simulator.
+    mu1/mu2 = 0.8 : rubber-track-on-concrete friction.
+    kp      = stiff contact (hard surface).
+    kd      = damping prevents bouncing at contact.
+    minDepth: small allowed interpenetration stabilises low-speed contact.
   -->
-  <!-- Chassis body — aluminium silver -->
-  <gazebo reference="base_link">
-    <material>Gazebo/Silver</material>
-  </gazebo>
-  <!-- Track pods — rubber black -->
-  <gazebo reference="front_left_track_link">
-    <material>Gazebo/DarkGrey</material>
-  </gazebo>
-  <gazebo reference="rear_left_track_link">
-    <material>Gazebo/DarkGrey</material>
-  </gazebo>
-  <gazebo reference="front_right_track_link">
-    <material>Gazebo/DarkGrey</material>
-  </gazebo>
-  <gazebo reference="rear_right_track_link">
-    <material>Gazebo/DarkGrey</material>
-  </gazebo>
-  <!-- Motor shafts — silver -->
-  <gazebo reference="front_motor_link">
-    <material>Gazebo/Silver</material>
-  </gazebo>
-  <gazebo reference="rear_motor_link">
-    <material>Gazebo/Silver</material>
-  </gazebo>
-  <!-- Electronics -->
-  <gazebo reference="raspberry_pi_link">
-    <material>Gazebo/Green</material>
-  </gazebo>
-  <gazebo reference="arduino_link">
-    <material>Gazebo/Blue</material>
-  </gazebo>
-  <gazebo reference="battery_link">
-    <material>Gazebo/Black</material>
-  </gazebo>
-  <gazebo reference="esp32_link">
-    <material>Gazebo/Blue</material>
-  </gazebo>
-  <gazebo reference="stm32_link">
-    <material>Gazebo/Red</material>
-  </gazebo>
-  <!-- Sensors -->
-  <gazebo reference="imu_link">
-    <material>Gazebo/Blue</material>
-  </gazebo>
-  <gazebo reference="downward_camera_link">
-    <material>Gazebo/DarkGrey</material>
-  </gazebo>
-  <gazebo reference="front_tof_link">
-    <material>Gazebo/Blue</material>
-  </gazebo>
-  <gazebo reference="front_left_tof_link">
-    <material>Gazebo/Blue</material>
-  </gazebo>
-  <gazebo reference="front_right_tof_link">
-    <material>Gazebo/Blue</material>
-  </gazebo>
-  <gazebo reference="rear_left_tof_link">
-    <material>Gazebo/Blue</material>
-  </gazebo>
-  <gazebo reference="rear_right_tof_link">
-    <material>Gazebo/Blue</material>
-  </gazebo>
+  <xacro:macro name="track_friction" params="link_name">
+    <gazebo reference="${link_name}">
+      <mu1>0.8</mu1>  <!-- longitudinal: grip for forward/back -->
+      <mu2>0.3</mu2>  <!-- lateral: LOW so tracks can skid-steer and TURN -->
+      <kp>1000000.0</kp>
+      <kd>100.0</kd>
+      <minDepth>0.001</minDepth>
+      <maxContacts>4</maxContacts>
+    </gazebo>
+  </xacro:macro>
+  <xacro:track_friction link_name="front_left_track_link"/>
+  <xacro:track_friction link_name="rear_left_track_link"/>
+  <xacro:track_friction link_name="front_right_track_link"/>
+  <xacro:track_friction link_name="rear_right_track_link"/>
+  <!-- ══ 7. Gazebo material colours ═══════════════════════════ -->
+  <gazebo reference="base_link">        <material>Gazebo/Silver</material>    </gazebo>
+  <gazebo reference="front_left_track_link">  <material>Gazebo/DarkGrey</material> </gazebo>
+  <gazebo reference="rear_left_track_link">   <material>Gazebo/DarkGrey</material> </gazebo>
+  <gazebo reference="front_right_track_link"> <material>Gazebo/DarkGrey</material> </gazebo>
+  <gazebo reference="rear_right_track_link">  <material>Gazebo/DarkGrey</material> </gazebo>
+  <gazebo reference="raspberry_pi_link"> <material>Gazebo/Green</material>    </gazebo>
+  <gazebo reference="arduino_link">      <material>Gazebo/Blue</material>     </gazebo>
+  <gazebo reference="battery_link">      <material>Gazebo/Black</material>    </gazebo>
+  <gazebo reference="esp32_link">        <material>Gazebo/Blue</material>     </gazebo>
+  <gazebo reference="stm32_link">        <material>Gazebo/Red</material>      </gazebo>
+  <gazebo reference="imu_link">          <material>Gazebo/Blue</material>     </gazebo>
+  <gazebo reference="downward_camera_link"> <material>Gazebo/DarkGrey</material> </gazebo>
+  <gazebo reference="front_tof_link">       <material>Gazebo/Blue</material>  </gazebo>
+  <gazebo reference="front_left_tof_link">  <material>Gazebo/Blue</material>  </gazebo>
+  <gazebo reference="front_right_tof_link"> <material>Gazebo/Blue</material>  </gazebo>
+  <gazebo reference="rear_left_tof_link">   <material>Gazebo/Blue</material>  </gazebo>
+  <gazebo reference="rear_right_tof_link">  <material>Gazebo/Blue</material>  </gazebo>
 </robot>

Commit message: teleop working

File: src/solarbot_description/urdf/base/chassis.xacro (robot description, xacro)
@@ -29,5 +29,5 @@
         lx="${track_full_length}"
         ly="${motor_shaft_length}"
-        lz="${track_pod_height}"/>
+        lz="0.084"/>
     </inertial>
     <!-- Central spine rail -->

File: src/solarbot_description/urdf/common/properties.xacro (robot description, xacro)
@@ -32,9 +32,9 @@
   <xacro:property name="track_y_offset"       value="0.078"/>
   <xacro:property name="track_z_offset"       value="-0.016"/>
-  <!-- ──  wheel (control) ──────────────────────────── -->
-  <xacro:property name="wheel_radius"         value="0.04"/>
+  <!-- ── Virtual wheel (control) ──────────────────────────── -->
+  <xacro:property name="wheel_radius"         value="0.040"/>
   <xacro:property name="wheel_width"          value="0.050"/>
   <xacro:property name="wheel_y_offset"       value="0.078"/>
-  <xacro:property name="wheel_mass"           value="0.0015"/>
+  <xacro:property name="wheel_mass"           value="0.01"/>
   <!-- ── Motors ───────────────────────────────────────────── -->
   <xacro:property name="motor_radius"         value="0.018"/>

File: src/solarbot_description/urdf/gazebo/gazebo.xacro (robot description, xacro)
@@ -16,5 +16,5 @@
       <right_joint>rear_right_wheel_joint</right_joint>
       <wheel_separation>0.156</wheel_separation>
-      <wheel_radius>0.04</wheel_radius>
+      <wheel_radius>0.040</wheel_radius>
       <odom_publish_frequency>30</odom_publish_frequency>
       <topic>cmd_vel</topic>
@@ -23,8 +23,8 @@
       <frame_id>odom</frame_id>
       <child_frame_id>base_footprint</child_frame_id>
-      <max_linear_acceleration>5.0</max_linear_acceleration>
-      <max_angular_acceleration>5.0</max_angular_acceleration>
-      <min_velocity>-1.0</min_velocity>
-      <max_velocity>1.0</max_velocity>
+      <max_linear_acceleration>0.5</max_linear_acceleration>
+      <max_angular_acceleration>1.0</max_angular_acceleration>
+      <min_velocity>-0.20</min_velocity>
+      <max_velocity>0.20</max_velocity>
     </plugin>
   </gazebo>
