Commit message: Description package updated

File: src/solarbot_description/urdf/base/chassis.xacro (robot description, xacro)
@@ -2,8 +2,5 @@
 <robot xmlns:xacro="http://www.ros.org/wiki/xacro">
   <!--
-    chassis.xacro  —  base_footprint + base_link frame only.
-    Track pods moved back to tracks.xacro (they are now real physics
-    objects). Motor shaft visuals remain inline here since they are
-    purely cosmetic with no physics role.
+    chassis.xacro — Fully enclosed, light-tight chassis body with original silver material
   -->
   <xacro:macro name="box_inertia" params="m lx ly lz">
@@ -12,4 +9,54 @@
       iyy="${m*(lx*lx + lz*lz)/12.0}" iyz="0"
       izz="${m*(lx*lx + ly*ly)/12.0}"/>
+  </xacro:macro>
+  <!-- Skirt wheel-cutout macro: splits what was a single continuous
+       skirt panel into 3 segments (front sliver / large middle piece /
+       rear sliver), leaving a gap at each wheel's X-position instead of
+       moving the skirt's Y-position outward. wheel_clearance gives a
+       small safety margin beyond the wheel's physical radius. -->
+  <xacro:property name="wheel_clearance" value="0.006"/>
+  <xacro:macro name="skirt_side" params="y_pos">
+    <!-- Front sliver: between front wheel's cutout and the chassis front edge -->
+    <visual>
+      <origin xyz="${(track_full_length/2 + track_front_x + wheel_radius + wheel_clearance)/2} ${y_pos} -0.010" rpy="0 0 0"/>
+      <geometry>
+        <box size="${track_full_length/2 - (track_front_x + wheel_radius + wheel_clearance)} 0.004 0.050"/>
+      </geometry>
+      <material name="silver"/>
+    </visual>
+    <collision>
+      <origin xyz="${(track_full_length/2 + track_front_x + wheel_radius + wheel_clearance)/2} ${y_pos} -0.010" rpy="0 0 0"/>
+      <geometry>
+        <box size="${track_full_length/2 - (track_front_x + wheel_radius + wheel_clearance)} 0.004 0.050"/>
+      </geometry>
+    </collision>
+    <!-- Middle: between the front and rear wheel cutouts -->
+    <visual>
+      <origin xyz="0 ${y_pos} -0.010" rpy="0 0 0"/>
+      <geometry>
+        <box size="${2*(track_front_x - wheel_radius - wheel_clearance)} 0.004 0.050"/>
+      </geometry>
+      <material name="silver"/>
+    </visual>
+    <collision>
+      <origin xyz="0 ${y_pos} -0.010" rpy="0 0 0"/>
+      <geometry>
+        <box size="${2*(track_front_x - wheel_radius - wheel_clearance)} 0.004 0.050"/>
+      </geometry>
+    </collision>
+    <!-- Rear sliver: mirror of the front sliver -->
+    <visual>
+      <origin xyz="${-(track_full_length/2 + track_front_x + wheel_radius + wheel_clearance)/2} ${y_pos} -0.010" rpy="0 0 0"/>
+      <geometry>
+        <box size="${track_full_length/2 - (track_front_x + wheel_radius + wheel_clearance)} 0.004 0.050"/>
+      </geometry>
+      <material name="silver"/>
+    </visual>
+    <collision>
+      <origin xyz="${-(track_full_length/2 + track_front_x + wheel_radius + wheel_clearance)/2} ${y_pos} -0.010" rpy="0 0 0"/>
+      <geometry>
+        <box size="${track_full_length/2 - (track_front_x + wheel_radius + wheel_clearance)} 0.004 0.050"/>
+      </geometry>
+    </collision>
   </xacro:macro>
   <!-- base_footprint — ground-plane projection, used by Nav2 -->
@@ -28,65 +75,42 @@
         m="${chassis_mass}"
         lx="${track_full_length}"
-        ly="${motor_shaft_length}"
+        ly="0.180"
         lz="0.084"/>
     </inertial>
-    <!-- Central spine rail -->
+    <!-- 1. MAIN SOLID CHASSIS ENCLOSURE (Fills space from bottom to top deck plate, 0 gaps) -->
     <visual>
-      <origin xyz="0 0 0" rpy="0 0 0"/>
+      <origin xyz="0 0 0.010" rpy="0 0 0"/>
       <geometry>
-        <box size="${chassis_rail_length} ${chassis_rail_width} ${chassis_rail_height}"/>
+        <box size="${track_full_length} 0.170 0.052"/>
       </geometry>
       <material name="silver"/>
     </visual>
     <collision>
-      <origin xyz="0 0 0" rpy="0 0 0"/>
+      <origin xyz="0 0 0.010" rpy="0 0 0"/>
       <geometry>
-        <box size="${chassis_rail_length} ${chassis_rail_width} ${chassis_rail_height}"/>
+        <box size="${track_full_length} 0.170 0.052"/>
       </geometry>
     </collision>
-    <!-- Front top plate -->
+    <!-- 2. FULL TOP LID DECK PLATE (Seals the top surface under electronics) -->
     <visual>
-      <origin xyz="${plate_length} 0 ${plate_z}" rpy="0 0 0"/>
+      <origin xyz="0 0 0.037" rpy="0 0 0"/>
       <geometry>
-        <box size="${plate_length} ${plate_width} ${plate_thickness}"/>
+        <box size="${track_full_length} 0.180 0.004"/>
       </geometry>
       <material name="silver"/>
     </visual>
     <collision>
-      <origin xyz="${plate_length} 0 ${plate_z}" rpy="0 0 0"/>
+      <origin xyz="0 0 0.037" rpy="0 0 0"/>
       <geometry>
-        <box size="${plate_length} ${plate_width} ${plate_thickness}"/>
+        <box size="${track_full_length} 0.180 0.004"/>
       </geometry>
     </collision>
-    <!-- Rear top plate -->
-    <visual>
-      <origin xyz="${-plate_length} 0 ${plate_z}" rpy="0 0 0"/>
-      <geometry>
-        <box size="${plate_length} ${plate_width} ${plate_thickness}"/>
-      </geometry>
-      <material name="silver"/>
-    </visual>
-    <collision>
-      <origin xyz="${-plate_length} 0 ${plate_z}" rpy="0 0 0"/>
-      <geometry>
-        <box size="${plate_length} ${plate_width} ${plate_thickness}"/>
-      </geometry>
-    </collision>
-    <!-- Left side rail (visual only) -->
-    <visual>
-      <origin xyz="0 ${side_rail_y} ${side_rail_z}" rpy="0 0 0"/>
-      <geometry>
-        <box size="${side_rail_length} ${side_rail_width} ${side_rail_height}"/>
-      </geometry>
-      <material name="silver"/>
-    </visual>
-    <!-- Right side rail (visual only) -->
-    <visual>
-      <origin xyz="0 ${-side_rail_y} ${side_rail_z}" rpy="0 0 0"/>
-      <geometry>
-        <box size="${side_rail_length} ${side_rail_width} ${side_rail_height}"/>
-      </geometry>
-      <material name="silver"/>
-    </visual>
+    <!-- 3. SIDE SKIRTING (Extends down along wheels to block side glare
+         into bottom camera) - Y position kept at 0.088 as originally
+         specified. Wheel interference resolved via cutouts (3 segments
+         per side, see skirt_side macro above) rather than moving the
+         skirt outward. -->
+    <xacro:skirt_side y_pos="0.088"/>
+    <xacro:skirt_side y_pos="-0.088"/>
     <!-- Front motor shaft (visual only) -->
     <visual>

File: src/solarbot_description/urdf/common/properties.xacro (robot description, xacro)
@@ -1,106 +1,87 @@
 <?xml version="1.0"?>
 <robot xmlns:xacro="http://www.ros.org/wiki/xacro">
-  <!--
-    properties.xacro
-    Single source of truth for ALL dimensions, masses and positions.
-    Edit numbers here — every other file picks them up automatically.
-    Real chassis measurements:
-      Total length : 393 mm
-      Total width  : 206 mm
-      Total height :  84 mm (tracks included)
-  -->
   <!-- ── Chassis body ──────────────────────────────────────── -->
-  <xacro:property name="chassis_rail_length"  value="0.270"/>
-  <xacro:property name="chassis_rail_width"   value="0.055"/>
-  <xacro:property name="chassis_rail_height"  value="0.022"/>
-  <xacro:property name="plate_length"         value="0.105"/>
-  <xacro:property name="plate_width"          value="0.145"/>
-  <xacro:property name="plate_thickness"      value="0.008"/>
-  <xacro:property name="plate_z"              value="0.034"/>
-  <xacro:property name="side_rail_length"     value="0.295"/>
-  <xacro:property name="side_rail_width"      value="0.014"/>
-  <xacro:property name="side_rail_height"     value="0.018"/>
-  <xacro:property name="side_rail_z"          value="-0.006"/>
-  <xacro:property name="side_rail_y"          value="0.070"/>
+  <xacro:property name="chassis_rail_length"   value="0.270"/>
+  <xacro:property name="chassis_rail_width"    value="0.055"/>
+  <xacro:property name="chassis_rail_height"   value="0.022"/>
+  <xacro:property name="plate_length"          value="0.105"/>
+  <xacro:property name="plate_width"           value="0.145"/>
+  <xacro:property name="plate_thickness"       value="0.008"/>
+  <xacro:property name="plate_z"               value="0.034"/>
+  <!-- ── Top Lid & Perimeter Skirting ──────────────────────── -->
+  <xacro:property name="lid_length"             value="0.393"/>
+  <xacro:property name="lid_width"              value="0.180"/>
+  <xacro:property name="lid_thickness"          value="0.004"/>
+  <xacro:property name="skirt_length"           value="0.380"/>
+  <xacro:property name="skirt_width"            value="0.170"/>
+  <xacro:property name="skirt_height"           value="0.030"/>
+  <xacro:property name="skirt_thickness"        value="0.003"/>
+  <xacro:property name="skirt_z_offset"         value="-0.020"/>
+  <xacro:property name="side_rail_length"      value="0.295"/>
+  <xacro:property name="side_rail_width"       value="0.014"/>
+  <xacro:property name="side_rail_height"      value="0.018"/>
+  <xacro:property name="side_rail_z"           value="-0.006"/>
+  <xacro:property name="side_rail_y"           value="0.070"/>
   <!-- ── Track geometry ───────────────────────────────────── -->
-  <xacro:property name="track_pod_length"     value="0.115"/>
-  <xacro:property name="track_pod_width"      value="0.050"/>
-  <xacro:property name="track_pod_height"     value="0.052"/>
-  <xacro:property name="track_full_length"    value="0.393"/>
-  <xacro:property name="track_front_x"        value="0.135"/>
-  <xacro:property name="track_rear_x"         value="-0.135"/>
-  <xacro:property name="track_y_offset"       value="0.078"/>
-  <xacro:property name="track_z_offset"       value="-0.016"/>
-  <!-- ── Virtual wheel (control) ──────────────────────────── -->
-  <xacro:property name="wheel_radius"         value="0.040"/>
-  <xacro:property name="wheel_width"          value="0.050"/>
-  <xacro:property name="wheel_y_offset"       value="0.078"/>
-  <xacro:property name="wheel_mass"           value="0.1"/>
+  <xacro:property name="track_pod_length"      value="0.115"/>
+  <xacro:property name="track_pod_width"       value="0.050"/>
+  <xacro:property name="track_pod_height"      value="0.052"/>
+  <xacro:property name="track_full_length"     value="0.393"/>
+  <xacro:property name="track_front_x"         value="0.135"/>
+  <xacro:property name="track_rear_x"          value="-0.135"/>
+  <xacro:property name="track_y_offset"        value="0.078"/>
+  <xacro:property name="track_z_offset"        value="-0.016"/>
+  <!-- ── Wheel ────────────────────────────────────────────── -->
+  <xacro:property name="wheel_radius"          value="0.040"/>
+  <xacro:property name="wheel_width"           value="0.050"/>
+  <xacro:property name="wheel_y_offset"        value="0.078"/>
+  <xacro:property name="wheel_mass"            value="0.1"/>
   <!-- ── Motors ───────────────────────────────────────────── -->
-  <xacro:property name="motor_radius"         value="0.018"/>
-  <xacro:property name="motor_shaft_length"   value="0.155"/>
-  <xacro:property name="motor_front_x"        value="0.155"/>
-  <xacro:property name="motor_z"              value="-0.006"/>
+  <xacro:property name="motor_radius"          value="0.018"/>
+  <xacro:property name="motor_shaft_length"    value="0.155"/>
+  <xacro:property name="motor_front_x"         value="0.155"/>
+  <xacro:property name="motor_z"               value="-0.006"/>
   <!-- ── Base heights ─────────────────────────────────────── -->
-  <xacro:property name="base_z_above_ground"  value="${wheel_radius}"/>
+  <xacro:property name="base_z_above_ground"   value="${wheel_radius}"/>
   <!-- ── Masses ────────────────────────────────────────────── -->
-  <xacro:property name="chassis_mass"         value="2.20"/>
-  <xacro:property name="track_pod_mass"       value="0.45"/>
-  <xacro:property name="virtual_wheel_mass"   value="0.001"/>
-  <!-- ══════════════════════════════════════════════════════ -->
-  <!-- ELECTRONICS POSITIONS                                 -->
-  <!-- All xyz relative to base_link origin.                 -->
-  <!-- Adjust once physical mounting is measured.            -->
-  <!-- ══════════════════════════════════════════════════════ -->
-  <!-- Battery pack (LiFePO4, centre-rear for balance) -->
-  <xacro:property name="battery_x"            value="-0.060"/>
-  <xacro:property name="battery_y"            value="0.000"/>
-  <xacro:property name="battery_z"            value="0.055"/>
-  <!-- Raspberry Pi 5 (rear top plate) -->
-  <xacro:property name="rpi_x"                value="-0.090"/>
-  <xacro:property name="rpi_y"                value="0.000"/>
-  <xacro:property name="rpi_z"                value="0.050"/>
-  <!-- ESP32 motor controller (front area, near motor driver) -->
-  <xacro:property name="esp32_x"              value="0.080"/>
-  <xacro:property name="esp32_y"              value="0.020"/>
-  <xacro:property name="esp32_z"              value="0.048"/>
-  <!-- STM32 safety controller (front top plate) -->
-  <xacro:property name="stm32_x"              value="0.080"/>
-  <xacro:property name="stm32_y"              value="-0.020"/>
-  <xacro:property name="stm32_z"              value="0.048"/>
-  <!-- ══════════════════════════════════════════════════════ -->
-  <!-- SENSOR POSITIONS                                      -->
-  <!-- All xyz relative to base_link origin.                 -->
-  <!-- ══════════════════════════════════════════════════════ -->
-  <!-- IMU (GY-91 / MPU9250 — centred on chassis) -->
-  <xacro:property name="imu_x"                value="0.000"/>
-  <xacro:property name="imu_y"                value="0.000"/>
-  <xacro:property name="imu_z"                value="0.045"/>
-  <!-- Downward camera (OV9732 — centre of chassis, looking down at panel) -->
-  <xacro:property name="camera_x"             value="0.000"/>
-  <xacro:property name="camera_y"             value="0.000"/>
-  <xacro:property name="camera_z"             value="-0.020"/>
-  <!-- Front obstacle ToF (forward-facing, above front edge) -->
-  <xacro:property name="front_tof_x"          value="0.200"/>
-  <xacro:property name="front_tof_y"          value="0.000"/>
-  <xacro:property name="front_tof_z"          value="0.010"/>
-  <!--
-    Corner cliff ToF sensors (downward-facing, detect panel edges).
-    Positioned just inboard of each track corner so they see the
-    panel surface drop-off before the wheels reach the edge.
-    rpy "0 1.5708 0" = pointing straight down (sensor board faces -z).
-    Adjust x/y offsets once physically mounted and tested.
-  -->
-  <xacro:property name="front_left_tof_x"     value="0.200"/>
-  <xacro:property name="front_left_tof_y"     value="0.075"/>
-  <xacro:property name="front_left_tof_z"     value="-0.010"/>
-  <xacro:property name="front_right_tof_x"    value="0.200"/>
-  <xacro:property name="front_right_tof_y"    value="-0.075"/>
-  <xacro:property name="front_right_tof_z"    value="-0.010"/>
-  <xacro:property name="rear_left_tof_x"      value="-0.200"/>
-  <xacro:property name="rear_left_tof_y"      value="0.075"/>
-  <xacro:property name="rear_left_tof_z"      value="-0.010"/>
-  <xacro:property name="rear_right_tof_x"     value="-0.200"/>
-  <xacro:property name="rear_right_tof_y"     value="-0.075"/>
-  <xacro:property name="rear_right_tof_z"     value="-0.010"/>
+  <xacro:property name="chassis_mass"          value="2.20"/>
+  <xacro:property name="track_pod_mass"        value="0.45"/>
+  <xacro:property name="virtual_wheel_mass"    value="0.001"/>
+  <!-- ── Electronics & Sensor Positions ─────────────────────── -->
+  <xacro:property name="battery_x"             value="-0.060"/>
+  <xacro:property name="battery_y"             value="0.000"/>
+  <xacro:property name="battery_z"             value="0.055"/>
+  <xacro:property name="rpi_x"                 value="-0.090"/>
+  <xacro:property name="rpi_y"                 value="0.000"/>
+  <xacro:property name="rpi_z"                 value="0.050"/>
+  <xacro:property name="esp32_x"               value="0.080"/>
+  <xacro:property name="esp32_y"               value="0.020"/>
+  <xacro:property name="esp32_z"               value="0.048"/>
+  <xacro:property name="stm32_x"               value="0.080"/>
+  <xacro:property name="stm32_y"               value="-0.020"/>
+  <xacro:property name="stm32_z"               value="0.048"/>
+  <xacro:property name="imu_x"                 value="0.000"/>
+  <xacro:property name="imu_y"                 value="0.000"/>
+  <xacro:property name="imu_z"                 value="0.045"/>
+  <xacro:property name="camera_x"              value="0.000"/>
+  <xacro:property name="camera_y"              value="0.000"/>
+  <xacro:property name="camera_z"              value="-0.020"/>
+  <xacro:property name="front_tof_x"           value="0.200"/>
+  <xacro:property name="front_tof_y"           value="0.000"/>
+  <xacro:property name="front_tof_z"           value="0.010"/>
+  <xacro:property name="front_left_tof_x"      value="0.200"/>
+  <xacro:property name="front_left_tof_y"      value="0.075"/>
+  <xacro:property name="front_left_tof_z"      value="-0.010"/>
+  <xacro:property name="front_right_tof_x"     value="0.200"/>
+  <xacro:property name="front_right_tof_y"     value="-0.075"/>
+  <xacro:property name="front_right_tof_z"     value="-0.010"/>
+  <xacro:property name="rear_left_tof_x"       value="-0.200"/>
+  <xacro:property name="rear_left_tof_y"       value="0.075"/>
+  <xacro:property name="rear_left_tof_z"       value="-0.010"/>
+  <xacro:property name="rear_right_tof_x"      value="-0.200"/>
+  <xacro:property name="rear_right_tof_y"      value="-0.075"/>
+  <xacro:property name="rear_right_tof_z"      value="-0.010"/>
+  <xacro:property name="gps_x"                 value="-0.090"/>
+  <xacro:property name="gps_y"                 value="0.000"/>
+  <xacro:property name="gps_z"                 value="0.055"/>
 </robot>

File: src/solarbot_description/urdf/gazebo/gazebo.xacro (robot description, xacro)
@@ -15,4 +15,20 @@
       <joint_name>rear_right_wheel_joint</joint_name>
       <topic>joint_states</topic>
+    </plugin>
+  </gazebo>
+  <!-- ══ 1b. Ground-truth odometry (SIM ONLY, for validation) ═══ -->
+  <!-- Publishes the model's actual world pose, unaffected by wheel
+       slip — this is the ground truth /odom_cam should be compared
+       against, matching the paper's evaluation method. Do NOT feed
+       this into any controller or EKF; it does not exist on real
+       hardware. -->
+  <gazebo>
+    <plugin filename="gz-sim-odometry-publisher-system"
+            name="gz::sim::systems::OdometryPublisher">
+      <odom_frame>ground_truth_odom</odom_frame>
+      <robot_base_frame>base_link</robot_base_frame>
+      <dimensions>3</dimensions>
+      <odom_publish_frequency>30</odom_publish_frequency>
+      <odom_topic>/ground_truth/odom</odom_topic>
     </plugin>
   </gazebo>
@@ -38,14 +54,41 @@
     </sensor>
   </gazebo>
+<!-- ══ GPS (NavSat) sensor ══════════════════════════════════ -->
+  <gazebo reference="gps_link">
+    <sensor name="gps_sensor" type="navsat">
+      <always_on>true</always_on>
+      <update_rate>10</update_rate>
+      <topic>/gps/fix</topic>
+      <gz_frame_id>gps_link</gz_frame_id>
+      <navsat>
+        <position_sensing>
+          <horizontal>
+            <noise type="gaussian">
+              <mean>0.0</mean>
+              <stddev>0.00001</stddev>  <!-- ~1.1 meter realistic GNSS noise -->
+            </noise>
+          </horizontal>
+          <vertical>
+            <noise type="gaussian">
+              <mean>0.0</mean>
+              <stddev>0.00002</stddev>  <!-- ~2.2 meter altitude noise -->
+            </noise>
+          </vertical>
+        </position_sensing>
+      </navsat>
+    </sensor>
+  </gazebo>
   <!-- ══ 3. Downward camera ═══════════════════════════════════ -->
   <gazebo reference="downward_camera_link">
     <sensor name="downward_camera" type="camera">
       <always_on>true</always_on>
-      <update_rate>30</update_rate>
+      <update_rate>40</update_rate>
+      <visualize>false</visualize>
       <topic>/camera/image_raw</topic>
-      <gz_frame_id>downward_camera_optical_frame</gz_frame_id>
-      <camera name="downward_camera">
-        <horizontal_fov>1.3614</horizontal_fov>
+      <camera>
+        <!-- OV9732 datasheet: 100 deg horizontal FOV = 1.74533 rad -->
+        <horizontal_fov>2.20</horizontal_fov>
         <image>
+           <!-- Native OV9732 resolution/aspect (16:9), matches USB listing -->
           <width>640</width>
           <height>480</height>
@@ -53,12 +96,7 @@
         </image>
         <clip>
-          <near>0.005</near>
-          <far>0.50</far>
+          <near>0.02</near>
+          <far>5.0</far>
         </clip>
-        <noise>
-          <type>gaussian</type>
-          <mean>0.0</mean>
-          <stddev>0.005</stddev>
-        </noise>
       </camera>
     </sensor>

File: src/solarbot_description/urdf/sensors/sensors.xacro (robot description, xacro)
@@ -72,8 +72,13 @@
     <visual>
       <geometry>
-        <box size="0.030 0.030 0.020"/>
+        <box size="0.032 0.032 0.022"/>
       </geometry>
       <material name="dark_gray"/>
     </visual>
+    <collision>
+      <geometry>
+        <box size="0.032 0.032 0.022"/>
+      </geometry>
+    </collision>
   </link>
   <joint name="downward_camera_joint" type="fixed">
@@ -88,10 +93,10 @@
     (Z forward = down into the panel, X right).
   -->
-  <link name="downward_camera_optical_frame"/>
+  <!-- <link name="downward_camera_optical_frame"/>
   <joint name="downward_camera_optical_joint" type="fixed">
     <parent link="downward_camera_link"/>
     <child  link="downward_camera_optical_frame"/>
-    <origin xyz="0 0 0" rpy="-1.5708 0 0"/>
-  </joint>
+    <origin xyz="0 0 0" rpy="-1.5708 0 -1.5708"/>
+  </joint> -->
   <!-- ── Front obstacle ToF (forward-facing) ───────────────── -->
   <!--
@@ -136,3 +141,17 @@
     z="${rear_right_tof_z}"
     rpy="0 1.5708 0"/>
+    <!-- ── GPS (UBX M8030 M8N) ───────────────────────────────── -->
+  <link name="gps_link">
+    <visual>
+      <geometry>
+        <cylinder radius="0.015" length="0.010"/>
+      </geometry>
+      <material name="blue"/>
+    </visual>
+  </link>
+  <joint name="gps_joint" type="fixed">
+    <parent link="base_link"/>
+    <child  link="gps_link"/>
+    <origin xyz="${gps_x} ${gps_y} ${gps_z}" rpy="0 0 0"/>
+  </joint>
 </robot>
