Commit message: Camera odom and map generation

File: src/solarbot_description/urdf/base/chassis.xacro (robot description, xacro)
@@ -2,5 +2,5 @@
 <robot xmlns:xacro="http://www.ros.org/wiki/xacro">
   <!--
-    chassis.xacro — Fully enclosed, light-tight chassis body with original silver material
+    chassis.xacro — Fully enclosed chassis body with side skirting and central camera shroud
   -->
   <xacro:macro name="box_inertia" params="m lx ly lz">
@@ -10,12 +10,8 @@
       izz="${m*(lx*lx + ly*ly)/12.0}"/>
   </xacro:macro>
-  <!-- Skirt wheel-cutout macro: splits what was a single continuous
-       skirt panel into 3 segments (front sliver / large middle piece /
-       rear sliver), leaving a gap at each wheel's X-position instead of
-       moving the skirt's Y-position outward. wheel_clearance gives a
-       small safety margin beyond the wheel's physical radius. -->
+  <!-- Skirt wheel-cutout macro: splits continuous skirt panel into 3 segments -->
   <xacro:property name="wheel_clearance" value="0.006"/>
   <xacro:macro name="skirt_side" params="y_pos">
-    <!-- Front sliver: between front wheel's cutout and the chassis front edge -->
+    <!-- Front sliver -->
     <visual>
       <origin xyz="${(track_full_length/2 + track_front_x + wheel_radius + wheel_clearance)/2} ${y_pos} -0.010" rpy="0 0 0"/>
@@ -31,5 +27,5 @@
       </geometry>
     </collision>
-    <!-- Middle: between the front and rear wheel cutouts -->
+    <!-- Middle piece -->
     <visual>
       <origin xyz="0 ${y_pos} -0.010" rpy="0 0 0"/>
@@ -45,5 +41,5 @@
       </geometry>
     </collision>
-    <!-- Rear sliver: mirror of the front sliver -->
+    <!-- Rear sliver -->
     <visual>
       <origin xyz="${-(track_full_length/2 + track_front_x + wheel_radius + wheel_clearance)/2} ${y_pos} -0.010" rpy="0 0 0"/>
@@ -78,5 +74,5 @@
         lz="0.084"/>
     </inertial>
-    <!-- 1. MAIN SOLID CHASSIS ENCLOSURE (Fills space from bottom to top deck plate, 0 gaps) -->
+    <!-- 1. MAIN SOLID CHASSIS ENCLOSURE -->
     <visual>
       <origin xyz="0 0 0.010" rpy="0 0 0"/>
@@ -92,5 +88,5 @@
       </geometry>
     </collision>
-    <!-- 2. FULL TOP LID DECK PLATE (Seals the top surface under electronics) -->
+    <!-- 2. FULL TOP LID DECK PLATE -->
     <visual>
       <origin xyz="0 0 0.037" rpy="0 0 0"/>
@@ -106,11 +102,71 @@
       </geometry>
     </collision>
-    <!-- 3. SIDE SKIRTING (Extends down along wheels to block side glare
-         into bottom camera) - Y position kept at 0.088 as originally
-         specified. Wheel interference resolved via cutouts (3 segments
-         per side, see skirt_side macro above) rather than moving the
-         skirt outward. -->
+    <!-- 3. SIDE SKIRTING -->
     <xacro:skirt_side y_pos="0.088"/>
     <xacro:skirt_side y_pos="-0.088"/>
+    <!-- 4. CAMERA SHROUD (Rectangular hood around the downward camera) -->
+    <xacro:property name="shroud_half_x" value="0.093"/>
+    <xacro:property name="shroud_half_y" value="0.036"/>
+    <xacro:property name="shroud_wall_t" value="0.003"/>
+    <xacro:property name="shroud_top_z" value="-0.005"/>
+    <xacro:property name="shroud_bottom_z" value="-0.038"/>
+    <xacro:property name="shroud_height" value="${shroud_top_z - shroud_bottom_z}"/>
+    <xacro:property name="shroud_center_z" value="${(shroud_top_z + shroud_bottom_z) / 2}"/>
+    <!-- Front wall -->
+    <visual>
+      <origin xyz="${camera_x + shroud_half_x} ${camera_y} ${shroud_center_z}" rpy="0 0 0"/>
+      <geometry>
+        <box size="${shroud_wall_t} ${shroud_half_y*2} ${shroud_height}"/>
+      </geometry>
+      <material name="dark_gray"/>
+    </visual>
+    <collision>
+      <origin xyz="${camera_x + shroud_half_x} ${camera_y} ${shroud_center_z}" rpy="0 0 0"/>
+      <geometry>
+        <box size="${shroud_wall_t} ${shroud_half_y*2} ${shroud_height}"/>
+      </geometry>
+    </collision>
+    <!-- Rear wall -->
+    <visual>
+      <origin xyz="${camera_x - shroud_half_x} ${camera_y} ${shroud_center_z}" rpy="0 0 0"/>
+      <geometry>
+        <box size="${shroud_wall_t} ${shroud_half_y*2} ${shroud_height}"/>
+      </geometry>
+      <material name="dark_gray"/>
+    </visual>
+    <collision>
+      <origin xyz="${camera_x - shroud_half_x} ${camera_y} ${shroud_center_z}" rpy="0 0 0"/>
+      <geometry>
+        <box size="${shroud_wall_t} ${shroud_half_y*2} ${shroud_height}"/>
+      </geometry>
+    </collision>
+    <!-- Left wall -->
+    <visual>
+      <origin xyz="${camera_x} ${camera_y + shroud_half_y} ${shroud_center_z}" rpy="0 0 0"/>
+      <geometry>
+        <box size="${shroud_half_x*2} ${shroud_wall_t} ${shroud_height}"/>
+      </geometry>
+      <material name="dark_gray"/>
+    </visual>
+    <collision>
+      <origin xyz="${camera_x} ${camera_y + shroud_half_y} ${shroud_center_z}" rpy="0 0 0"/>
+      <geometry>
+        <box size="${shroud_half_x*2} ${shroud_wall_t} ${shroud_height}"/>
+      </geometry>
+    </collision>
+    <!-- Right wall -->
+    <visual>
+      <origin xyz="${camera_x} ${camera_y - shroud_half_y} ${shroud_center_z}" rpy="0 0 0"/>
+      <geometry>
+        <box size="${shroud_half_x*2} ${shroud_wall_t} ${shroud_height}"/>
+      </geometry>
+      <material name="dark_gray"/>
+    </visual>
+    <collision>
+      <origin xyz="${camera_x} ${camera_y - shroud_half_y} ${shroud_center_z}" rpy="0 0 0"/>
+      <geometry>
+        <box size="${shroud_half_x*2} ${shroud_wall_t} ${shroud_height}"/>
+      </geometry>
+    </collision>
     <!-- Front motor shaft (visual only) -->
     <visual>

File: src/solarbot_description/urdf/common/properties.xacro (robot description, xacro)
@@ -13,75 +13,73 @@
   <xacro:property name="lid_width"              value="0.180"/>
   <xacro:property name="lid_thickness"          value="0.004"/>
-  <xacro:property name="skirt_length"           value="0.380"/>
-  <xacro:property name="skirt_width"            value="0.170"/>
-  <xacro:property name="skirt_height"           value="0.030"/>
-  <xacro:property name="skirt_thickness"        value="0.003"/>
-  <xacro:property name="skirt_z_offset"         value="-0.020"/>
-  <xacro:property name="side_rail_length"      value="0.295"/>
-  <xacro:property name="side_rail_width"       value="0.014"/>
-  <xacro:property name="side_rail_height"      value="0.018"/>
-  <xacro:property name="side_rail_z"           value="-0.006"/>
-  <xacro:property name="side_rail_y"           value="0.070"/>
+  <xacro:property name="side_rail_length"       value="0.295"/>
+  <xacro:property name="side_rail_width"        value="0.014"/>
+  <xacro:property name="side_rail_height"       value="0.018"/>
+  <xacro:property name="side_rail_z"            value="-0.006"/>
+  <xacro:property name="side_rail_y"            value="0.070"/>
   <!-- ── Track geometry ───────────────────────────────────── -->
-  <xacro:property name="track_pod_length"      value="0.115"/>
-  <xacro:property name="track_pod_width"       value="0.050"/>
-  <xacro:property name="track_pod_height"      value="0.052"/>
-  <xacro:property name="track_full_length"     value="0.393"/>
-  <xacro:property name="track_front_x"         value="0.135"/>
-  <xacro:property name="track_rear_x"          value="-0.135"/>
-  <xacro:property name="track_y_offset"        value="0.078"/>
-  <xacro:property name="track_z_offset"        value="-0.016"/>
+  <xacro:property name="track_pod_length"       value="0.115"/>
+  <xacro:property name="track_pod_width"        value="0.050"/>
+  <xacro:property name="track_pod_height"       value="0.052"/>
+  <xacro:property name="track_full_length"      value="0.393"/>
+  <xacro:property name="track_front_x"          value="0.135"/>
+  <xacro:property name="track_rear_x"           value="-0.135"/>
+  <xacro:property name="track_y_offset"         value="0.078"/>
+  <xacro:property name="track_z_offset"         value="-0.016"/>
   <!-- ── Wheel ────────────────────────────────────────────── -->
-  <xacro:property name="wheel_radius"          value="0.040"/>
-  <xacro:property name="wheel_width"           value="0.050"/>
-  <xacro:property name="wheel_y_offset"        value="0.078"/>
-  <xacro:property name="wheel_mass"            value="0.1"/>
+  <xacro:property name="wheel_radius"           value="0.040"/>
+  <xacro:property name="wheel_width"            value="0.050"/>
+  <xacro:property name="wheel_y_offset"         value="0.078"/>
+  <xacro:property name="wheel_mass"             value="0.1"/>
+  <!-- ── Inboard Skirting Calculation ────────────────────── -->
+  <!-- Inner boundary for central camera shroud (~0.051m) -->
+  <xacro:property name="skirt_inboard_y"       value="${wheel_y_offset - (wheel_width/2) - 0.002}"/>
   <!-- ── Motors ───────────────────────────────────────────── -->
-  <xacro:property name="motor_radius"          value="0.018"/>
-  <xacro:property name="motor_shaft_length"    value="0.155"/>
-  <xacro:property name="motor_front_x"         value="0.155"/>
-  <xacro:property name="motor_z"               value="-0.006"/>
+  <xacro:property name="motor_radius"           value="0.018"/>
+  <xacro:property name="motor_shaft_length"     value="0.155"/>
+  <xacro:property name="motor_front_x"          value="0.155"/>
+  <xacro:property name="motor_z"                value="-0.006"/>
   <!-- ── Base heights ─────────────────────────────────────── -->
-  <xacro:property name="base_z_above_ground"   value="${wheel_radius}"/>
+  <xacro:property name="base_z_above_ground"    value="${wheel_radius}"/>
   <!-- ── Masses ────────────────────────────────────────────── -->
-  <xacro:property name="chassis_mass"          value="2.20"/>
-  <xacro:property name="track_pod_mass"        value="0.45"/>
-  <xacro:property name="virtual_wheel_mass"    value="0.001"/>
+  <xacro:property name="chassis_mass"           value="2.20"/>
+  <xacro:property name="track_pod_mass"         value="0.45"/>
+  <xacro:property name="virtual_wheel_mass"     value="0.001"/>
   <!-- ── Electronics & Sensor Positions ─────────────────────── -->
-  <xacro:property name="battery_x"             value="-0.060"/>
-  <xacro:property name="battery_y"             value="0.000"/>
-  <xacro:property name="battery_z"             value="0.055"/>
-  <xacro:property name="rpi_x"                 value="-0.090"/>
-  <xacro:property name="rpi_y"                 value="0.000"/>
-  <xacro:property name="rpi_z"                 value="0.050"/>
-  <xacro:property name="esp32_x"               value="0.080"/>
-  <xacro:property name="esp32_y"               value="0.020"/>
-  <xacro:property name="esp32_z"               value="0.048"/>
-  <xacro:property name="stm32_x"               value="0.080"/>
-  <xacro:property name="stm32_y"               value="-0.020"/>
-  <xacro:property name="stm32_z"               value="0.048"/>
-  <xacro:property name="imu_x"                 value="0.000"/>
-  <xacro:property name="imu_y"                 value="0.000"/>
-  <xacro:property name="imu_z"                 value="0.045"/>
-  <xacro:property name="camera_x"              value="0.000"/>
-  <xacro:property name="camera_y"              value="0.000"/>
-  <xacro:property name="camera_z"              value="-0.020"/>
-  <xacro:property name="front_tof_x"           value="0.200"/>
-  <xacro:property name="front_tof_y"           value="0.000"/>
-  <xacro:property name="front_tof_z"           value="0.010"/>
-  <xacro:property name="front_left_tof_x"      value="0.200"/>
-  <xacro:property name="front_left_tof_y"      value="0.075"/>
-  <xacro:property name="front_left_tof_z"      value="-0.010"/>
-  <xacro:property name="front_right_tof_x"     value="0.200"/>
-  <xacro:property name="front_right_tof_y"     value="-0.075"/>
-  <xacro:property name="front_right_tof_z"     value="-0.010"/>
-  <xacro:property name="rear_left_tof_x"       value="-0.200"/>
-  <xacro:property name="rear_left_tof_y"       value="0.075"/>
-  <xacro:property name="rear_left_tof_z"       value="-0.010"/>
-  <xacro:property name="rear_right_tof_x"      value="-0.200"/>
-  <xacro:property name="rear_right_tof_y"      value="-0.075"/>
-  <xacro:property name="rear_right_tof_z"      value="-0.010"/>
-  <xacro:property name="gps_x"                 value="-0.090"/>
-  <xacro:property name="gps_y"                 value="0.000"/>
-  <xacro:property name="gps_z"                 value="0.055"/>
+  <xacro:property name="battery_x"              value="-0.060"/>
+  <xacro:property name="battery_y"              value="0.000"/>
+  <xacro:property name="battery_z"              value="0.055"/>
+  <xacro:property name="rpi_x"                  value="-0.090"/>
+  <xacro:property name="rpi_y"                  value="0.000"/>
+  <xacro:property name="rpi_z"                  value="0.050"/>
+  <xacro:property name="esp32_x"                value="0.080"/>
+  <xacro:property name="esp32_y"                value="0.020"/>
+  <xacro:property name="esp32_z"                value="0.048"/>
+  <xacro:property name="stm32_x"                value="0.080"/>
+  <xacro:property name="stm32_y"                value="-0.020"/>
+  <xacro:property name="stm32_z"                value="0.048"/>
+  <xacro:property name="imu_x"                  value="0.000"/>
+  <xacro:property name="imu_y"                  value="0.000"/>
+  <xacro:property name="imu_z"                  value="0.045"/>
+  <xacro:property name="camera_x"               value="0.000"/>
+  <xacro:property name="camera_y"               value="0.000"/>
+  <xacro:property name="camera_z"               value="-0.020"/>
+  <xacro:property name="front_tof_x"            value="0.200"/>
+  <xacro:property name="front_tof_y"            value="0.000"/>
+  <xacro:property name="front_tof_z"            value="0.010"/>
+  <xacro:property name="front_left_tof_x"       value="0.200"/>
+  <xacro:property name="front_left_tof_y"       value="0.075"/>
+  <xacro:property name="front_left_tof_z"       value="-0.010"/>
+  <xacro:property name="front_right_tof_x"      value="0.200"/>
+  <xacro:property name="front_right_tof_y"      value="-0.075"/>
+  <xacro:property name="front_right_tof_z"      value="-0.010"/>
+  <xacro:property name="rear_left_tof_x"        value="-0.200"/>
+  <xacro:property name="rear_left_tof_y"        value="0.075"/>
+  <xacro:property name="rear_left_tof_z"        value="-0.010"/>
+  <xacro:property name="rear_right_tof_x"       value="-0.200"/>
+  <xacro:property name="rear_right_tof_y"       value="-0.075"/>
+  <xacro:property name="rear_right_tof_z"       value="-0.010"/>
+  <xacro:property name="gps_x"                  value="-0.090"/>
+  <xacro:property name="gps_y"                  value="0.000"/>
+  <xacro:property name="gps_z"                  value="0.055"/>
 </robot>
