Commit message: Add initial robot description and RViz visualization

File: src/solarbot_description/urdf/common/properties.xacro (robot description, xacro)
@@ -22,5 +22,5 @@
   <!-- ========================================================= -->
   <!-- Initial estimate -->
-  <xacro:property name="robot_mass" value="5.0"/>
+  <xacro:property name="robot_mass" value="5.5"/>
   <!-- ========================================================= -->
   <!-- SENSOR POSITIONS                                           -->

Commit message: teleop working

File: src/solarbot_description/urdf/common/properties.xacro (robot description, xacro)
@@ -32,7 +32,9 @@
   <xacro:property name="track_y_offset"       value="0.078"/>
   <xacro:property name="track_z_offset"       value="-0.016"/>
-  <!-- ── Virtual wheel (control) ──────────────────────────── -->
-  <xacro:property name="wheel_radius"         value="0.026"/>
+  <!-- ──  wheel (control) ──────────────────────────── -->
+  <xacro:property name="wheel_radius"         value="0.04"/>
   <xacro:property name="wheel_width"          value="0.050"/>
+  <xacro:property name="wheel_y_offset"       value="0.078"/>
+  <xacro:property name="wheel_mass"           value="0.0015"/>
   <!-- ── Motors ───────────────────────────────────────────── -->
   <xacro:property name="motor_radius"         value="0.018"/>

File: src/solarbot_description/urdf/gazebo/gazebo.xacro (robot description, xacro)
@@ -16,5 +16,5 @@
       <right_joint>rear_right_wheel_joint</right_joint>
       <wheel_separation>0.156</wheel_separation>
-      <wheel_radius>0.026</wheel_radius>
+      <wheel_radius>0.04</wheel_radius>
       <odom_publish_frequency>30</odom_publish_frequency>
       <topic>cmd_vel</topic>
@@ -23,8 +23,8 @@
       <frame_id>odom</frame_id>
       <child_frame_id>base_footprint</child_frame_id>
-      <max_linear_acceleration>0.5</max_linear_acceleration>
-      <max_angular_acceleration>1.0</max_angular_acceleration>
-      <min_velocity>-0.15</min_velocity>
-      <max_velocity>0.15</max_velocity>
+      <max_linear_acceleration>5.0</max_linear_acceleration>
+      <max_angular_acceleration>5.0</max_angular_acceleration>
+      <min_velocity>-1.0</min_velocity>
+      <max_velocity>1.0</max_velocity>
     </plugin>
   </gazebo>
@@ -147,14 +147,13 @@
     </sensor>
   </gazebo>
-  <!-- ══ 6. Track pod friction (all four pods) ════════════════ -->
-  <!--
-    mu1/mu2 = 0.8 : rubber-track-on-concrete friction.
-    kp      = stiff contact (hard surface).
-    kd      = damping prevents bouncing at contact.
-    minDepth: small allowed interpenetration stabilises low-speed contact.
-  -->
-  <xacro:macro name="track_friction" params="link_name">
+  <!-- ══ 6. Wheel friction ════════════════════════════════════ -->
+<!--
+  mu1 = 0.9  : longitudinal (forward/back grip)
+  mu2 = 0.3  : lateral (lower = allows skid-steer turning)
+  kp/kd      : stiff hard-surface contact
+-->
+  <xacro:macro name="wheel_friction" params="link_name">
     <gazebo reference="${link_name}">
-      <mu1>0.8</mu1>  <!-- longitudinal: grip for forward/back -->
+      <mu1>0.9</mu1>  <!-- longitudinal: grip for forward/back -->
       <mu2>0.3</mu2>  <!-- lateral: LOW so tracks can skid-steer and TURN -->
       <kp>1000000.0</kp>
@@ -164,14 +163,14 @@
     </gazebo>
   </xacro:macro>
-  <xacro:track_friction link_name="front_left_track_link"/>
-  <xacro:track_friction link_name="rear_left_track_link"/>
-  <xacro:track_friction link_name="front_right_track_link"/>
-  <xacro:track_friction link_name="rear_right_track_link"/>
+  <xacro:wheel_friction link_name="front_left_wheel_link"/>
+  <xacro:wheel_friction link_name="rear_left_wheel_link"/>
+  <xacro:wheel_friction link_name="front_right_wheel_link"/>
+  <xacro:wheel_friction link_name="rear_right_wheel_link"/>
   <!-- ══ 7. Gazebo material colours ═══════════════════════════ -->
   <gazebo reference="base_link">        <material>Gazebo/Silver</material>    </gazebo>
-  <gazebo reference="front_left_track_link">  <material>Gazebo/DarkGrey</material> </gazebo>
-  <gazebo reference="rear_left_track_link">   <material>Gazebo/DarkGrey</material> </gazebo>
-  <gazebo reference="front_right_track_link"> <material>Gazebo/DarkGrey</material> </gazebo>
-  <gazebo reference="rear_right_track_link">  <material>Gazebo/DarkGrey</material> </gazebo>
+  <gazebo reference="front_left_wheel_link">  <material>Gazebo/DarkGrey</material> </gazebo>
+  <gazebo reference="rear_left_wheel_link">   <material>Gazebo/DarkGrey</material> </gazebo>
+  <gazebo reference="front_right_wheel_link"> <material>Gazebo/DarkGrey</material> </gazebo>
+  <gazebo reference="rear_right_wheel_link">  <material>Gazebo/DarkGrey</material> </gazebo>
   <gazebo reference="raspberry_pi_link"> <material>Gazebo/Green</material>    </gazebo>
   <gazebo reference="arduino_link">      <material>Gazebo/Blue</material>     </gazebo>

File: src/solarbot_description/urdf/solarbot.urdf.xacro (robot description, xacro)
@@ -19,5 +19,5 @@
   <!-- ── 2. Base ───────────────────────────────────────────────── -->
   <xacro:include filename="$(find solarbot_description)/urdf/base/chassis.xacro"/>
-  <xacro:include filename="$(find solarbot_description)/urdf/base/tracks.xacro"/>
+  <xacro:include filename="$(find solarbot_description)/urdf/base/wheels.xacro"/>
   <!-- ── 3. Sensors ────────────────────────────────────────────── -->
   <xacro:include filename="$(find solarbot_description)/urdf/sensors/sensors.xacro"/>

Commit message: Perimeter following complete

File: src/solarbot_description/urdf/common/properties.xacro (robot description, xacro)
@@ -36,5 +36,5 @@
   <xacro:property name="wheel_width"          value="0.050"/>
   <xacro:property name="wheel_y_offset"       value="0.078"/>
-  <xacro:property name="wheel_mass"           value="0.01"/>
+  <xacro:property name="wheel_mass"           value="0.1"/>
   <!-- ── Motors ───────────────────────────────────────────── -->
   <xacro:property name="motor_radius"         value="0.018"/>
@@ -89,18 +89,18 @@
     Positioned just inboard of each track corner so they see the
     panel surface drop-off before the wheels reach the edge.
-    rpy "0 0 0" = pointing straight down (sensor board faces -z).
+    rpy "0 1.5708 0" = pointing straight down (sensor board faces -z).
     Adjust x/y offsets once physically mounted and tested.
   -->
-  <xacro:property name="front_left_tof_x"     value="0.170"/>
-  <xacro:property name="front_left_tof_y"     value="0.065"/>
+  <xacro:property name="front_left_tof_x"     value="0.200"/>
+  <xacro:property name="front_left_tof_y"     value="0.075"/>
   <xacro:property name="front_left_tof_z"     value="-0.010"/>
-  <xacro:property name="front_right_tof_x"    value="0.170"/>
-  <xacro:property name="front_right_tof_y"    value="-0.065"/>
+  <xacro:property name="front_right_tof_x"    value="0.200"/>
+  <xacro:property name="front_right_tof_y"    value="-0.075"/>
   <xacro:property name="front_right_tof_z"    value="-0.010"/>
-  <xacro:property name="rear_left_tof_x"      value="-0.170"/>
-  <xacro:property name="rear_left_tof_y"      value="0.065"/>
+  <xacro:property name="rear_left_tof_x"      value="-0.200"/>
+  <xacro:property name="rear_left_tof_y"      value="0.075"/>
   <xacro:property name="rear_left_tof_z"      value="-0.010"/>
-  <xacro:property name="rear_right_tof_x"     value="-0.170"/>
-  <xacro:property name="rear_right_tof_y"     value="-0.065"/>
+  <xacro:property name="rear_right_tof_x"     value="-0.200"/>
+  <xacro:property name="rear_right_tof_y"     value="-0.075"/>
   <xacro:property name="rear_right_tof_z"     value="-0.010"/>
 </robot>

File: src/solarbot_description/urdf/gazebo/gazebo.xacro (robot description, xacro)
@@ -127,6 +127,7 @@
   <xacro:macro name="wheel_friction" params="link_name">
     <gazebo reference="${link_name}">
-      <mu1>0.9</mu1>  <!-- longitudinal: grip for forward/back -->
-      <mu2>0.3</mu2>  <!-- lateral: LOW so tracks can skid-steer and TURN -->
+      <mu1>0.9</mu1><!-- longitudinal: grip for forward/back -->
+      <mu2>0.2</mu2>
+      <fdir1>1 0 0 </fdir1>
       <kp>1000000.0</kp>
       <kd>100.0</kd>

File: src/solarbot_description/urdf/sensors/sensors.xacro (robot description, xacro)
@@ -80,5 +80,5 @@
     <parent link="base_link"/>
     <child  link="downward_camera_link"/>
-    <origin xyz="${camera_x} ${camera_y} ${camera_z}" rpy="0 0 0"/>
+    <origin xyz="${camera_x} ${camera_y} ${camera_z}" rpy="0 1.5708 0"/>
   </joint>
   <!--
@@ -92,9 +92,9 @@
     <parent link="downward_camera_link"/>
     <child  link="downward_camera_optical_frame"/>
-    <origin xyz="0 0 -0.020" rpy="-1.5708 0 -1.5708"/>
+    <origin xyz="0 0 0" rpy="-1.5708 0 0"/>
   </joint>
   <!-- ── Front obstacle ToF (forward-facing) ───────────────── -->
   <!--
-    rpy="0 1.5708 0" tilts the sensor to face forward (+X direction).
+    rpy="0 0 0" tilts the sensor to face forward (+X direction).
     Detects obstacles ahead of the robot on the panel surface.
   -->
@@ -104,8 +104,8 @@
     y="${front_tof_y}"
     z="${front_tof_z}"
-    rpy="0 1.5708 0"/>
+    rpy="0 0 0"/>
   <!-- ── Corner cliff ToF sensors (downward-facing) ────────── -->
   <!--
-    rpy="0 0 0" — sensor faces straight down (-Z in base_link frame).
+    rpy="0 1.5708 0" — sensor faces straight down (-Z in base_link frame).
     Placed at the four corners just inboard of the tracks so they
     detect the panel edge drop-off before wheels reach it.
@@ -117,5 +117,5 @@
     y="${front_left_tof_y}"
     z="${front_left_tof_z}"
-    rpy="0 0 0"/>
+    rpy="0 1.5708 0"/>
   <xacro:tof_sensor
     name="front_right_tof"
@@ -123,5 +123,5 @@
     y="${front_right_tof_y}"
     z="${front_right_tof_z}"
-    rpy="0 0 0"/>
+    rpy="0 1.5708 0"/>
   <xacro:tof_sensor
     name="rear_left_tof"
@@ -129,5 +129,5 @@
     y="${rear_left_tof_y}"
     z="${rear_left_tof_z}"
-    rpy="0 0 0"/>
+    rpy="0 1.5708 0"/>
   <xacro:tof_sensor
     name="rear_right_tof"
@@ -135,4 +135,4 @@
     y="${rear_right_tof_y}"
     z="${rear_right_tof_z}"
-    rpy="0 0 0"/>
+    rpy="0 1.5708 0"/>
 </robot>
