Commit message: TOF positioning changed

File: src/solarbot_description/urdf/common/properties.xacro (robot description, xacro)
@@ -22,5 +22,5 @@
   <xacro:property name="track_pod_width"        value="0.050"/>
   <xacro:property name="track_pod_height"       value="0.052"/>
-  <xacro:property name="track_full_length"      value="0.393"/>
+  <xacro:property name="track_full_length"       value="0.393"/>
   <xacro:property name="track_front_x"          value="0.135"/>
   <xacro:property name="track_rear_x"           value="-0.135"/>
@@ -33,5 +33,4 @@
   <xacro:property name="wheel_mass"             value="0.1"/>
   <!-- ── Inboard Skirting Calculation ────────────────────── -->
-  <!-- Inner boundary for central camera shroud (~0.051m) -->
   <xacro:property name="skirt_inboard_y"       value="${wheel_y_offset - (wheel_width/2) - 0.002}"/>
   <!-- ── Motors ───────────────────────────────────────────── -->
@@ -65,19 +64,17 @@
   <xacro:property name="camera_y"               value="0.000"/>
   <xacro:property name="camera_z"               value="-0.020"/>
-  <xacro:property name="front_tof_x"            value="0.200"/>
-  <xacro:property name="front_tof_y"            value="0.000"/>
-  <xacro:property name="front_tof_z"            value="0.010"/>
-  <xacro:property name="front_left_tof_x"       value="0.200"/>
-  <xacro:property name="front_left_tof_y"       value="0.075"/>
-  <xacro:property name="front_left_tof_z"       value="-0.010"/>
-  <xacro:property name="front_right_tof_x"      value="0.200"/>
-  <xacro:property name="front_right_tof_y"      value="-0.075"/>
-  <xacro:property name="front_right_tof_z"      value="-0.010"/>
-  <xacro:property name="rear_left_tof_x"        value="-0.200"/>
-  <xacro:property name="rear_left_tof_y"        value="0.075"/>
-  <xacro:property name="rear_left_tof_z"        value="-0.010"/>
-  <xacro:property name="rear_right_tof_x"       value="-0.200"/>
-  <xacro:property name="rear_right_tof_y"       value="-0.075"/>
-  <xacro:property name="rear_right_tof_z"       value="-0.010"/>
+  <xacro:property name="front_mid_tof_x"        value="0.200"/>
+  <xacro:property name="front_mid_tof_y"        value="0.000"/>
+  <xacro:property name="front_mid_tof_z"        value="-0.010"/>
+  <xacro:property name="rear_mid_tof_x"         value="-0.200"/>
+  <xacro:property name="rear_mid_tof_y"         value="0.000"/>
+  <xacro:property name="rear_mid_tof_z"         value="-0.010"/>
+  <xacro:property name="left_mid_tof_x"         value="0.000"/>
+  <xacro:property name="left_mid_tof_y"         value="0.115"/>
+  <xacro:property name="left_mid_tof_z"         value="-0.010"/>
+  <!-- Right side: VL53L5CX grid sensor -->
+  <xacro:property name="right_mid_tof_x"        value="0.000"/>
+  <xacro:property name="right_mid_tof_y"        value="-0.105"/>
+  <xacro:property name="right_mid_tof_z"        value="-0.005"/>
   <xacro:property name="gps_x"                  value="-0.090"/>
   <xacro:property name="gps_y"                  value="0.000"/>

File: src/solarbot_description/urdf/gazebo/gazebo.xacro (robot description, xacro)
@@ -131,31 +131,72 @@
     </gazebo>
   </xacro:macro>
-  <xacro:cliff_tof_gazebo link_name="front_left_tof_link"   topic="/front_left_tof"/>
-  <xacro:cliff_tof_gazebo link_name="front_right_tof_link" topic="/front_right_tof"/>
-  <xacro:cliff_tof_gazebo link_name="rear_left_tof_link"    topic="/rear_left_tof"/>
-  <xacro:cliff_tof_gazebo link_name="rear_right_tof_link"   topic="/rear_right_tof"/>
-  <!-- ══ 5. Front obstacle ToF ════════════════════════════════ -->
-  <gazebo reference="front_tof_link">
-    <sensor name="front_tof_sensor" type="gpu_lidar">
+  <xacro:cliff_tof_gazebo link_name="front_mid_tof_link" topic="/front_mid_tof"/>
+  <xacro:cliff_tof_gazebo link_name="rear_mid_tof_link"  topic="/rear_mid_tof"/>
+  <xacro:cliff_tof_gazebo link_name="left_mid_tof_link"  topic="/left_mid_tof"/>
+  <!-- ══ 5. Right side grid ToF (VL53L5CX-class, simulated approximation) ═ -->
+  <!-- Real sensor: genuine 8x8=64-ray grid. This block now matches that
+       directly - 8 horizontal x 8 vertical samples, both spanning
+       +/-22.98deg (per-axis FOV derived from the confirmed real 65deg
+       diagonal FOV, same method the VL53L5CX-BNO08X-viewer firmware's
+       own config.py uses). This gives Gazebo's own ray visualization
+       and physics a true square-spreading fan, matching the real
+       sensor's reference visualization - NOT the earlier 64x1
+       flattened-single-row approximation, which looked like a flat
+       line/wedge instead of a square.
+       STILL UNVERIFIED: whether ros_gz_bridge's LaserScan converter
+       correctly carries through BOTH dimensions to ROS's
+       sensor_msgs/LaserScan, which has no vertical field at all. Gazebo's
+       own internal gz.msgs.LaserScan CAN represent 2D scan data, but the
+       ROS-side message fundamentally cannot - the bridge's actual
+       behavior with a genuinely 2D input (rather than 1D) needs
+       confirming empirically once this is running, not assumed.
+       CHECK THIS FIRST once built: run "ros2 topic echo /right_mid_tof
+       once" (single dash flag, not shown literally here since XML
+       comments can't contain double-dash sequences)
+       - does `ranges` contain all 64 values, or does something look
+       wrong/truncated/only-one-row? If the bridge mishandles the 2D
+       input, the fallback is switching this sensor to publish
+       PointCloud2 instead (which natively supports 2D structure) and
+       updating solarbot_perimeter_node.py's parsing to match - a real
+       scope increase, not attempted here, but the correct fix if the
+       LaserScan bridge turns out not to work cleanly.
+       Range 0.020-4.000m matches config.py's real MIN_RANGE_MM/
+       MAX_RANGE_MM exactly. Orientation (down + outward tilt) is
+       inherited automatically from right_mid_tof_link's joint in
+       sensors.xacro - not configured here.
+       NOTE: the 4m max range above is a sensor ceiling, not a
+       guarantee of reach - actual horizontal reach into the panel
+       gaps is set by mount height + tilt angle (see the reach-vs-tilt
+       derivation on the right_mid_tof instantiation in sensors.xacro).
+       With the current 30.6deg-below-horizontal boresight and 5cm
+       mount height, the grid's rows reach roughly 3.8-35cm depending
+       on row, nowhere near 4m - that's expected and correct for
+       resolving a 0.3-0.5m gap up close, not a sign of something
+       wrong with the range config here. -->
+  <gazebo reference="right_mid_tof_link">
+    <sensor name="right_mid_tof_sensor" type="gpu_lidar">
       <always_on>true</always_on>
       <update_rate>50</update_rate>
-      <topic>/front_tof</topic>
-      <gz_frame_id>front_tof_link</gz_frame_id>
+      <topic>/right_mid_tof</topic>
+      <gz_frame_id>right_mid_tof_link</gz_frame_id>
       <lidar>
         <scan>
           <horizontal>
-            <samples>1</samples><resolution>1</resolution>
-            <min_angle>0</min_angle><max_angle>0</max_angle>
+            <samples>8</samples><resolution>1</resolution>
+            <min_angle>-0.4011</min_angle><max_angle>0.4011</max_angle>
           </horizontal>
           <vertical>
-            <samples>1</samples><resolution>1</resolution>
-            <min_angle>0</min_angle><max_angle>0</max_angle>
+            <samples>8</samples><resolution>1</resolution>
+            <min_angle>-0.4011</min_angle><max_angle>0.4011</max_angle>
           </vertical>
         </scan>
         <range>
-          <min>0.010</min><max>2.000</max><resolution>0.001</resolution>
+          <!-- Confirmed real datasheet values (VL53L5CX-BNO08X-viewer
+               firmware's config.py: MIN_RANGE_MM=20, MAX_RANGE_MM=4000),
+               not estimates. -->
+          <min>0.020</min><max>4.000</max><resolution>0.001</resolution>
         </range>
         <noise>
-          <type>gaussian</type><mean>0.0</mean><stddev>0.003</stddev>
+          <type>gaussian</type><mean>0.0</mean><stddev>0.002</stddev>
         </noise>
       </lidar>
@@ -191,8 +232,7 @@
   <gazebo reference="imu_link">          <material>Gazebo/Blue</material>     </gazebo>
   <gazebo reference="downward_camera_link"> <material>Gazebo/DarkGrey</material> </gazebo>
-  <gazebo reference="front_tof_link">       <material>Gazebo/Blue</material>  </gazebo>
-  <gazebo reference="front_left_tof_link">  <material>Gazebo/Blue</material>  </gazebo>
-  <gazebo reference="front_right_tof_link"> <material>Gazebo/Blue</material>  </gazebo>
-  <gazebo reference="rear_left_tof_link">   <material>Gazebo/Blue</material>  </gazebo>
-  <gazebo reference="rear_right_tof_link">  <material>Gazebo/Blue</material>  </gazebo>
+  <gazebo reference="front_mid_tof_link">   <material>Gazebo/Blue</material>  </gazebo>
+  <gazebo reference="rear_mid_tof_link">    <material>Gazebo/Blue</material>  </gazebo>
+  <gazebo reference="left_mid_tof_link">    <material>Gazebo/Blue</material>  </gazebo>
+  <gazebo reference="right_mid_tof_link">   <material>Gazebo/DarkGrey</material>  </gazebo>
 </robot>

File: src/solarbot_description/urdf/sensors/sensors.xacro (robot description, xacro)
@@ -9,15 +9,15 @@
       downward_camera_link        OV9732 downward-facing camera
       downward_camera_optical_frame  ROS optical frame (Z forward, X right)
-      front_tof_link              Forward obstacle ToF
-      front_left_tof_link  }
-      front_right_tof_link }      Corner cliff ToF sensors
-      rear_left_tof_link   }      (detect panel edges, face downward)
-      rear_right_tof_link  }
+      front_mid_tof_link          Point ToF (VL53L0X), front side
+      rear_mid_tof_link           Point ToF (VL53L0X), rear side
+      left_mid_tof_link           Point ToF (VL53L0X), left side
+      right_mid_tof_link          Grid ToF (VL53L5CX), right side -
+                                   actively used for continuous lateral
+                                   edge-following, not just trip/stop
     Published ROS topics (driver nodes, not defined here):
       /imu
       /camera/image_raw
-      /front_tof
-      /front_left_tof   /front_right_tof
-      /rear_left_tof    /rear_right_tof
+      /front_mid_tof   /rear_mid_tof
+      /left_mid_tof    /right_mid_tof
     All positions come from common/properties.xacro.
     NOTE — camera optical frame rotation:
@@ -54,4 +54,23 @@
     </joint>
   </xacro:macro>
+  <!-- Grid ToF (VL53L5CX-class multi-zone sensor) - larger box than the
+       point sensors, purely visual distinction so it's identifiable in
+       RViz/Gazebo. Update the box size once real board dimensions are
+       confirmed - currently a placeholder estimate (~25x25mm breakout). -->
+  <xacro:macro name="grid_tof_sensor" params="name x y z rpy">
+    <link name="${name}_link">
+      <visual>
+        <geometry>
+          <box size="0.025 0.025 0.008"/>
+        </geometry>
+        <material name="dark_gray"/>
+      </visual>
+    </link>
+    <joint name="${name}_joint" type="fixed">
+      <parent link="base_link"/>
+      <child  link="${name}_link"/>
+      <origin xyz="${x} ${y} ${z}" rpy="${rpy}"/>
+    </joint>
+  </xacro:macro>
   <!-- ── IMU ───────────────────────────────────────────────── -->
   <link name="imu_link">
@@ -99,47 +118,83 @@
     <origin xyz="0 0 0" rpy="-1.5708 0 -1.5708"/>
   </joint> -->
-  <!-- ── Front obstacle ToF (forward-facing) ───────────────── -->
-  <!--
-    rpy="0 0 0" tilts the sensor to face forward (+X direction).
-    Detects obstacles ahead of the robot on the panel surface.
+  <!-- ── Middle-of-side ToF sensors ─────────────────────────── -->
+  <!--
+    Replaces the earlier front + 4-corner layout entirely. One sensor
+    centered on each side. front/rear/left are point sensors
+    (VL53L0X-class); right is a VL53L5CX-class grid sensor, actively
+    used for continuous lateral edge-following in
+    solarbot_perimeter_node.py (not just a trip-and-stop reading like
+    the others).
+    front_mid / rear_mid: trigger the "reached the end of this side"
+    stop-and-turn event, same role the old front_tof/corner sensors
+    played, just repositioned.
+    left_mid: passive point sensor, safety backup only.
+    right_mid (GRID): tilted 35deg OUTWARD from straight-down (toward
+    -Y, across the gap) rather than forward along the direction of
+    travel - lets it see the panel edge on the far side of the gap
+    (the next panel over), not just the current edge beneath the robot.
+    See the detailed rpy derivation comment at its instantiation below.
   -->
   <xacro:tof_sensor
-    name="front_tof"
-    x="${front_tof_x}"
-    y="${front_tof_y}"
-    z="${front_tof_z}"
-    rpy="0 0 0"/>
-  <!-- ── Corner cliff ToF sensors (downward-facing) ────────── -->
-  <!--
-    rpy="0 1.5708 0" — sensor faces straight down (-Z in base_link frame).
-    Placed at the four corners just inboard of the tracks so they
-    detect the panel edge drop-off before wheels reach it.
-    These feed edge_guard_node to trigger the safety stop + turn.
-  -->
-  <xacro:tof_sensor
-    name="front_left_tof"
-    x="${front_left_tof_x}"
-    y="${front_left_tof_y}"
-    z="${front_left_tof_z}"
+    name="front_mid_tof"
+    x="${front_mid_tof_x}"
+    y="${front_mid_tof_y}"
+    z="${front_mid_tof_z}"
     rpy="0 1.5708 0"/>
   <xacro:tof_sensor
-    name="front_right_tof"
-    x="${front_right_tof_x}"
-    y="${front_right_tof_y}"
-    z="${front_right_tof_z}"
+    name="rear_mid_tof"
+    x="${rear_mid_tof_x}"
+    y="${rear_mid_tof_y}"
+    z="${rear_mid_tof_z}"
     rpy="0 1.5708 0"/>
   <xacro:tof_sensor
-    name="rear_left_tof"
-    x="${rear_left_tof_x}"
-    y="${rear_left_tof_y}"
-    z="${rear_left_tof_z}"
+    name="left_mid_tof"
+    x="${left_mid_tof_x}"
+    y="${left_mid_tof_y}"
+    z="${left_mid_tof_z}"
     rpy="0 1.5708 0"/>
-  <xacro:tof_sensor
-    name="rear_right_tof"
-    x="${rear_right_tof_x}"
-    y="${rear_right_tof_y}"
-    z="${rear_right_tof_z}"
-    rpy="0 1.5708 0"/>
-    <!-- ── GPS (UBX M8030 M8N) ───────────────────────────────── -->
+  <!-- right_mid_tof tilt: pitch=0.534 (30.6deg) + yaw=-1.5708 (-90deg)
+       combine to tilt the downward beam OUTWARD toward -Y (right side,
+       across the gap toward the next panel), not forward along the
+       direction of travel. Roll has no effect on this sensor's final
+       beam direction (its default scan axis is local +X, which is
+       invariant under any roll rotation applied before the pitch) -
+       the outward tilt is achieved through pitch+yaw composition
+       instead.
+       REACH FIX (was pitch=0.9599 / 55deg): at the old 55deg-below-
+       horizontal tilt and a 3cm mount height, horizontal reach before
+       hitting a surface is only height*cot(elevation) ~= 0.03*0.70 =
+       2.1cm - nowhere near the 0.3-0.5m panel gaps, so every ray in
+       the grid was hitting the near-flush gap floor marker almost
+       immediately instead of the neighboring panel. This was NOT a
+       sensor-range limitation (max range is still 4m, see gazebo.xacro)
+       - it was mount height + tilt angle geometry.
+       New boresight: 30.6deg below horizontal, paired with
+       right_mid_tof_z raised to +0.010 in properties.xacro (5cm mount
+       height instead of 3cm). With the sensor's +/-22.5deg per-axis
+       FOV (see gazebo.xacro sensor block) this spreads the 8x8 grid's
+       rows across:
+         top row    (30.6-22.5=8.1deg below horizontal):  5cm*cot(8.1)  ~= 0.35m reach -> clears the 0.3m row gap, hits next panel
+         boresight  (30.6deg):                             5cm*cot(30.6)~= 0.084m reach
+         bottom row (30.6+22.5=53.1deg below horizontal):  5cm*cot(53.1)~= 0.038m reach -> still tight enough for near gap-floor/cliff read
+       Top-row hits are a grazing ~8deg intercept on a ~1.2cm-tall
+       target from 35cm away - fragile to mount height/pitch/roll
+       tolerance while driving. Prefer treating "top rows near max-range
+       + bottom rows showing gap floor" as the CROSS_GAP signature in
+       solarbot_roof_coverage_node.py rather than requiring a clean top-
+       row panel hit every cycle. If more margin is needed, raising
+       mount height further is a bigger lever than tightening the angle
+       more. Verified numerically: final beam direction with the new
+       pitch is (0, -0.861, -0.509) - shallower down (was -0.819,
+       now -0.509 in z) and more outward-leaning (was -0.574, now
+       -0.861 in y) than before, which is exactly the trade that buys
+       the extra horizontal reach. -->
+  <xacro:grid_tof_sensor
+    name="right_mid_tof"
+    x="${right_mid_tof_x}"
+    y="${right_mid_tof_y}"
+    z="${right_mid_tof_z}"
+    rpy="0 0.534 -1.5708"/>
+  <!-- ── GPS (UBX M8030 M8N) ───────────────────────────────── -->
   <link name="gps_link">
     <visual>
