Commit message: Nav2 params updated

File: src/solarbot_description/urdf/control/ros2_control.xacro (robot description, xacro)
@@ -13,5 +13,5 @@
     <hardware>
       <xacro:if value="$(arg use_real_hardware)">
-        <plugin>panelbot_hardware/SkidSteerHardware</plugin>
+        <plugin>diffdrive_arduino/DiffDriveArduinoHardware</plugin>
         <param name="serial_port">$(arg serial_port)</param>
         <param name="baud_rate">115200</param>

File: src/solarbot_description/urdf/gazebo/gazebo.xacro (robot description, xacro)
@@ -219,20 +219,3 @@
   <xacro:wheel_friction link_name="front_right_wheel_link"/>
   <xacro:wheel_friction link_name="rear_right_wheel_link"/>
-  <!-- ══ 7. Gazebo material colours ═══════════════════════════ -->
-  <gazebo reference="base_link">        <material>Gazebo/Silver</material>    </gazebo>
-  <gazebo reference="front_left_wheel_link">  <material>Gazebo/DarkGrey</material> </gazebo>
-  <gazebo reference="rear_left_wheel_link">   <material>Gazebo/DarkGrey</material> </gazebo>
-  <gazebo reference="front_right_wheel_link"> <material>Gazebo/DarkGrey</material> </gazebo>
-  <gazebo reference="rear_right_wheel_link">  <material>Gazebo/DarkGrey</material> </gazebo>
-  <gazebo reference="raspberry_pi_link"> <material>Gazebo/Green</material>    </gazebo>
-  <gazebo reference="arduino_link">      <material>Gazebo/Blue</material>     </gazebo>
-  <gazebo reference="battery_link">      <material>Gazebo/Black</material>    </gazebo>
-  <gazebo reference="esp32_link">        <material>Gazebo/Blue</material>     </gazebo>
-  <gazebo reference="stm32_link">        <material>Gazebo/Red</material>      </gazebo>
-  <gazebo reference="imu_link">          <material>Gazebo/Blue</material>     </gazebo>
-  <gazebo reference="downward_camera_link"> <material>Gazebo/DarkGrey</material> </gazebo>
-  <gazebo reference="front_mid_tof_link">   <material>Gazebo/Blue</material>  </gazebo>
-  <gazebo reference="rear_mid_tof_link">    <material>Gazebo/Blue</material>  </gazebo>
-  <gazebo reference="left_mid_tof_link">    <material>Gazebo/Blue</material>  </gazebo>
-  <gazebo reference="right_mid_tof_link">   <material>Gazebo/DarkGrey</material>  </gazebo>
 </robot>
